Commit message: Moveit 6dof plugin generate

File: src/mobile_manipulator/model/mobile_manipulatornoJplate.xacro (robot description, xacro)
@@ -436,5 +436,5 @@
   <xacro:FxdJoint id="SQ2_AXB2B" trans="0 0 0" parent="square_plate_2" child="AXB2B_SQ_Y" />
   <xacro:FxdJoint id="AXB2B_Y" trans="0 0.07 0.055" parent="AXB2B_SQ_Y" child="wrist_yaw_motor" />
-  <xacro:Revjoint id="wrist yaw" trans="0 -0.0035 -0.0150" rpy="0 3.14 0" parent="wrist_yaw_motor" child="AXBrak_Y_R" axis="0 0 1" l="-2" u="+2" v="1.0"/>
+  <xacro:Revjoint id="wrist_yaw" trans="0 -0.0035 -0.0150" rpy="0 3.14 0" parent="wrist_yaw_motor" child="AXBrak_Y_R" axis="0 0 1" l="-2" u="+2" v="1.0"/>
   <xacro:FxdJoint id="AXBYR_R" trans="0 0 0" parent="AXBrak_Y_R" child="wrist_roll_motor"/>
   <xacro:Revjoint id="wrist_roll" trans="0 0.0 0.0409163" rpy="0 3.14 0" parent="wrist_roll_motor" child="gripper" axis="0 1 0" l="-2" u="+2" v="1.0"/>

File: src/mobile_manipulator/model/mobile_manipulatornojplate.urdf (robot description, URDF)
Before this commit: robot mobile_manipulator, 16 links, 16 joints
Joints:
- removed joint wrist yaw
- added joint wrist_yaw: type revolute, parent wrist_yaw_motor, child AXBrak_Y_R, origin xyz=0 -0.0035 -0.0150 rpy=0 3.14 0, axis 0 0 1, limit lower=-2 upper=+2 effort=30 velocity=1.0
