Commit message: .dae file generated

File: src/mobile_manipulator/model/mobile_manipulator.urdf (robot description, URDF)
Before this commit: robot mobile_manipulator, 16 links, 16 joints
Links:
- removed link square_plate_2
Joints:
- removed joint SQ2_AXB2B
- removed joint WP_SQ2
- joint shoulder_pitch: origin xyz=0 0 0.035 rpy=0 0 0 -> xyz=0 0 0.035 rpy=0 0.0 0

File: src/mobile_manipulator/model/mobile_manipulator.xacro (robot description, xacro)
@@ -399,9 +399,9 @@
     <xacro:square_plate_Collision trans="0.02 -0.0156 0.0737" rpy="3.14 1.57 -1.57"/>
   </link>
-    <link name="square_plate_2">
+    <!--link name="square_plate_2">
     <xacro:square_plate_Inertial trans="-0.02 -0.0156 0.0737" rpy="3.14 1.57 -1.57"/>
     <xacro:square_plate_Visual trans="-0.02 -0.0156 0.0737" rpy="3.14 1.57 -1.57"/>
     <xacro:square_plate_Collision trans="-0.02 -0.0156 0.0737" rpy="3.14 1.57 -1.57"/>
-  </link>
+  </link-->
   <link name="AXB2B_SQ_Y">
     <xacro:AxBack_Inertial trans="0.02 0.048 0.0737" rpy="0 1.57 3.14"/>
@@ -424,5 +424,5 @@
   <xacro:Revjoint id="shoulder_yaw" trans="0 0.188 0.2577" rpy="0 0 3.14" parent="shoulder_yaw_motor" child="shoulder_bracket" axis="0 0 1" l="-3.0357" u="3.24426" v="1.0"/>
   <!-- 0 0 0.025 -->
-  <xacro:Revjoint id="shoulder_pitch" trans="0 0 0.035" rpy="0 0 0" parent="shoulder_bracket" child="shoulder_pitch_motor" axis="1 0 0" l="-1.973232422" u="1.916503906" v="1.0"/>
+  <xacro:Revjoint id="shoulder_pitch" trans="0 0 0.035" rpy="0 0.0 0" parent="shoulder_bracket" child="shoulder_pitch_motor" axis="1 0 0" l="-1.973232422" u="1.916503906" v="1.0"/>
   <xacro:FxdJoint id="s1_l2" trans="0 0 0" parent="shoulder_pitch_motor" child="biscep"/>
   <xacro:FxdJoint id="l2_l2B" trans="0 0 0" parent="biscep" child="elbow_bracket"/>
@@ -432,7 +432,5 @@
   <xacro:Revjoint id="wrist_pitch" trans="0 0 ${length + 0.052 + 0.054}" rpy="0 0 0" parent="wrist_bracket" child="wrist_pitch_motor" axis="1 0 0" l="-2.36344086" u="2.368556533" v="1.0"/>
   <xacro:FxdJoint id="WP_SQ1" trans="0 0 0" parent="wrist_pitch_motor" child="square_plate_1" />
-  <xacro:FxdJoint id="WP_SQ2" trans="0 0 0" parent="wrist_pitch_motor" child="square_plate_2" />
   <xacro:FxdJoint id="SQ1_AXB2B" trans="0 0 0" parent="square_plate_1" child="AXB2B_SQ_Y" />
-  <xacro:FxdJoint id="SQ2_AXB2B" trans="0 0 0" parent="square_plate_2" child="AXB2B_SQ_Y" />
   <xacro:FxdJoint id="AXB2B_Y" trans="0 0.07 0.055" parent="AXB2B_SQ_Y" child="wrist_yaw_motor" />
   <xacro:Revjoint id="wrist_yaw" trans="0 -0.0035 -0.0150" rpy="0 3.14 0" parent="wrist_yaw_motor" child="AXBrak_Y_R" axis="0 0 1" l="-2" u="+2" v="1.0"/>

Commit message: URDF changed: rotation along Zaxis

File: src/mobile_manipulator/model/mobile_manipulator.urdf (robot description, URDF)
Before this commit: robot mobile_manipulator, 15 links, 14 joints
Joints:
- joint elbow: axis 1 0 0 -> 0 0 1; origin xyz=0 0 0.186 rpy=0 0 0 -> xyz=0.186 0 0 rpy=0 0 0
- joint shoulder_pitch: axis 1 0 0 -> 0 0 1; origin xyz=0 0 0.035 rpy=0 0.0 0 -> xyz=0 0 0.035 rpy=0 -1.57 0.0
- joint wrist_pitch: axis 1 0 0 -> 0 0 1; origin xyz=0 0 0.202 rpy=0 0 0 -> xyz=0.202 0 0  rpy=0 0 0
- joint wrist_roll: axis 0 1 0 -> 0 0 1; origin xyz=0 0.0 0.0409163 rpy=0 3.14 0 -> xyz=0 0.0 0.0409163 rpy=-1.57 3.14 0
- joint wrist_yaw: origin xyz=0 -0.0035 -0.0150 rpy=0 3.14 0 -> xyz=0.04 0 -0.055 rpy=0 -1.57 0

File: src/mobile_manipulator/model/mobile_manipulator.xacro (robot description, xacro)
@@ -345,42 +345,42 @@
   </link>
   <link name="shoulder_pitch_motor">
-    <xacro:MXInertial trans="0 0 0" rpy="1.57 -3.14 1.57"/>
-    <xacro:MXVisual trans="0 0 0" rpy="1.57 -3.14 1.57"/>
-    <xacro:MXCollision_dual_motor trans="0 0 0" rpy="1.57 -3.14 1.57"/>
+    <xacro:MXInertial trans="0 0 0" rpy="0 0 1.57"/>
+    <xacro:MXVisual trans="0 0 0" rpy="0.0 0.0 1.57"/>
+    <xacro:MXCollision_dual_motor trans="0 0 0" rpy="0 0 1.57"/>
   </link>
   <link name="biscep">
-    <xacro:LinkInertial trans="0 0 ${0.051+(length/2)}" rpy="0 0 0" />
-    <xacro:LinkVisual trans="0 0 ${0.051+(length/2)}" rpy="0 0 0" />
-    <xacro:LinkCollision trans="0 0 ${0.051+(length/2)}" rpy="0 0 0" />
+    <xacro:LinkInertial trans="${0.051+(length/2)} 0 0" rpy="0 1.57 0" />
+    <xacro:LinkVisual trans="${0.051+(length/2)} 0 0" rpy="0 1.57 0" />
+    <xacro:LinkCollision trans="${0.051+(length/2)} 0 0" rpy="0 1.57 0" />
   </link>
   <link name="elbow_bracket">
-    <xacro:BracketInertial trans="0 0 ${0.052+length}" rpy="0 3.14 0"/>
-    <xacro:BracketVisual trans="0 0 ${0.052+length}" rpy="0 3.14 0"/>
-    <xacro:BracketCollision trans="0 0 ${0.052+length}" rpy="0 3.14 0"/>
+    <xacro:BracketInertial trans="${0.052+length} 0 0" rpy="0 -1.57 0"/>
+    <xacro:BracketVisual trans="${0.052+length} 0 0" rpy="0 -1.57 0"/>
+    <xacro:BracketCollision trans="${0.052+length} 0 0" rpy="0 -1.57 0"/>
   </link>
   <link name="elbow_motor">
-    <xacro:MXInertial trans="0 0 0" rpy="1.57 0 0"/>
-    <xacro:MXVisual trans="0 0 0" rpy="1.57 3.14 -1.57"/>
-    <xacro:MXCollision trans="0 0 0" rpy="1.57 3.14 -1.57"/>
+    <xacro:MXInertial trans="0 0 0" rpy="0 0 1.57"/>
+    <xacro:MXVisual trans="0 0 0" rpy="0 0 1.57"/>
+    <xacro:MXCollision trans="0  0 0" rpy="0 0 1.57"/>
   </link>
   <link name="forearm">
-    <xacro:LinkInertial trans="0 0 ${0.052+(length/2)}" rpy="0 0 0" />
-    <xacro:LinkVisual trans="0 0 ${0.052+(length/2)}" rpy="0 0 0" />
-    <xacro:LinkCollision trans="0 0 ${0.052+(length/2)}" rpy="0 0 0" />
+    <xacro:LinkInertial trans="${0.052+(length/2)} 0 0" rpy="0 1.57 0" />
+    <xacro:LinkVisual trans="${0.052+(length/2)} 0 0" rpy="0 1.57 0" />
+    <xacro:LinkCollision trans="${0.052+(length/2)} 0 0" rpy="0 1.57 0" />
   </link>
   <link name="wrist_bracket">
-    <xacro:AxBracketInertial trans="0 0 ${0.052+length+0.054}" rpy="1.57 0 1.57"/>
-    <xacro:AxBracketVisual trans="0 0 ${0.052+length+0.054}" rpy="1.57 0 1.57"/>
-    <xacro:AxBracketCollision trans="0 0 ${0.052+length+0.054}" rpy="1.57 0 1.57"/>
+    <xacro:AxBracketInertial trans="${0.052+length+0.054} 0 0" rpy="0 0 -1.57"/>
+    <xacro:AxBracketVisual trans="${0.052+length+0.054} 0 0" rpy="0 0 -1.57"/>
+    <xacro:AxBracketCollision trans="${0.052+length+0.054} 0 0" rpy="0 0 -1.57"/>
   </link>
   <link name="wrist_pitch_motor">
-    <xacro:AXInertial trans="0 0 0" rpy="-1.57 0 -1.57"/>
-    <xacro:AXVisual trans="0 0 0" rpy="-1.57 0 -1.57"/>
-    <xacro:AXCollision trans="0 0 0" rpy="-1.57 0 -1.57"/>
+    <xacro:AXInertial trans="0 0 0" rpy="0 0 1.57"/>
+    <xacro:AXVisual trans="0 0 0" rpy="0 0 1.57"/>
+    <xacro:AXCollision trans="0 0 0" rpy="0 0 1.57"/>
   </link>
   <link name="wrist_yaw_motor">
-    <xacro:AXInertial trans="0 0.0 0.0" rpy="0 0 0"/>
-    <xacro:AXVisual trans="0 0.0 0.0" rpy="0 3.14 0"/>
-    <xacro:AXCollision trans="0 0.0 0.0" rpy="0 3.14 0"/>
+    <xacro:AXInertial trans="0.055 0.0 -0.056" rpy="0 1.57 0"/>
+    <xacro:AXVisual trans="0.055 0.0 -0.056" rpy="0 1.57 0"/>
+    <xacro:AXCollision trans="0.055 0.0 -0.056" rpy="0 1.57 0"/>
   </link>
   <link name="wrist_roll_motor">
@@ -395,7 +395,7 @@
   </link-->
   <link name="square_plate_1">
-    <xacro:square_plate_Inertial trans="0.02 -0.0156 0.0737" rpy="3.14 1.57 -1.57"/>
-    <xacro:square_plate_Visual trans="0.02 -0.0156 0.0737" rpy="3.14 1.57 -1.57"/>
-    <xacro:square_plate_Collision trans="0.02 -0.0156 0.0737" rpy="3.14 1.57 -1.57"/>
+    <xacro:square_plate_Inertial trans="0.035 -0.0156 0.02" rpy="-1.57 0 0"/>
+    <xacro:square_plate_Visual trans="0.035 -0.0156 0.02" rpy="-1.57 0 0"/>
+    <xacro:square_plate_Collision trans="0.035 -0.0156 0.0" rpy="-1.57 0 0"/>
   </link>
     <!--link name="square_plate_2">
@@ -405,7 +405,7 @@
   </link-->
   <link name="AXB2B_SQ_Y">
-    <xacro:AxBack_Inertial trans="0.02 0.048 0.0737" rpy="0 1.57 3.14"/>
-    <xacro:AxBack_Visual trans="0.02 0.048 0.0737" rpy="0 1.57 3.14"/>
-    <xacro:AxBack_Collision trans="0.02 0.048 0.0737" rpy="0 1.57 3.14"/>
+    <xacro:AxBack_Inertial trans="0.0737 0.048 -0.02" rpy="0 0 3.14"/>
+    <xacro:AxBack_Visual trans="0.0737 0.048 -0.02" rpy="0 0 3.14"/>
+    <xacro:AxBack_Collision trans="0.0737 0.048 -0.02" rpy="0 0 3.14"/>
   </link>
   <link name="AXBrak_Y_R">
@@ -415,7 +415,7 @@
   </link>
  <link name ="gripper">
-    <xacro:gripper_Inertial trans="0.007654 0.085866 -0.03272" rpy="-3.14 3.14 -3.14"/>
-    <xacro:gripper_Visual trans="0.007654 0.085866 -0.03272" rpy="-3.14 3.14 -3.14"/>
-    <xacro:gripper_Collision trans="0.007654 0.085866 -0.03272" rpy="-3.14 3.14 -3.14"/>
+    <xacro:gripper_Inertial trans="0.006 0.035 0.085" rpy="1.57 0 0"/>
+    <xacro:gripper_Visual trans="0.006 0.035 0.085" rpy="1.57 0 0"/>
+    <xacro:gripper_Collision trans="0.006 0.035 0.085" rpy="1.57 0 0"/>
   </link>
   <!-- 0.0812 -->
@@ -424,17 +424,17 @@
   <xacro:Revjoint id="shoulder_yaw" trans="0 0.188 0.2577" rpy="0 0 3.14" parent="shoulder_yaw_motor" child="shoulder_bracket" axis="0 0 1" l="-3.0357" u="3.24426" v="1.0"/>
   <!-- 0 0 0.025 -->
-  <xacro:Revjoint id="shoulder_pitch" trans="0 0 0.035" rpy="0 0.0 0" parent="shoulder_bracket" child="shoulder_pitch_motor" axis="1 0 0" l="-1.973232422" u="1.916503906" v="1.0"/>
+  <xacro:Revjoint id="shoulder_pitch" trans="0 0 0.035" rpy="0 -1.57 0.0" parent="shoulder_bracket" child="shoulder_pitch_motor" axis="0 0 1" l="-1.973232422" u="1.916503906" v="1.0"/>
   <xacro:FxdJoint id="s1_l2" trans="0 0 0" parent="shoulder_pitch_motor" child="biscep"/>
   <xacro:FxdJoint id="l2_l2B" trans="0 0 0" parent="biscep" child="elbow_bracket"/>
-  <xacro:Revjoint id="elbow" trans="0 0 ${0.052 + (length) + 0.038}" rpy="0 0 0" parent="elbow_bracket" child="elbow_motor" axis="1 0 0" l="-1.99" u="1.971699219" v="1.0"/>
+  <xacro:Revjoint id="elbow" trans="${0.052 + (length) + 0.038} 0 0" rpy="0 0 0" parent="elbow_bracket" child="elbow_motor" axis="0 0 1" l="-1.99" u="1.971699219" v="1.0"/>
   <xacro:FxdJoint id="e_l3" trans="0 0 0" parent="elbow_motor" child="forearm"/>
   <xacro:FxdJoint id="l3_l3B" trans="0 0 0" parent="forearm" child="wrist_bracket"/>
-  <xacro:Revjoint id="wrist_pitch" trans="0 0 ${length + 0.052 + 0.054}" rpy="0 0 0" parent="wrist_bracket" child="wrist_pitch_motor" axis="1 0 0" l="-2.36344086" u="2.368556533" v="1.0"/>
+  <xacro:Revjoint id="wrist_pitch" trans="${length + 0.052 + 0.054} 0 0 " rpy="0 0 0" parent="wrist_bracket" child="wrist_pitch_motor" axis="0 0 1" l="-2.36344086" u="2.368556533" v="1.0"/>
   <xacro:FxdJoint id="WP_SQ1" trans="0 0 0" parent="wrist_pitch_motor" child="square_plate_1" />
   <xacro:FxdJoint id="SQ1_AXB2B" trans="0 0 0" parent="square_plate_1" child="AXB2B_SQ_Y" />
   <xacro:FxdJoint id="AXB2B_Y" trans="0 0.07 0.055" parent="AXB2B_SQ_Y" child="wrist_yaw_motor" />
-  <xacro:Revjoint id="wrist_yaw" trans="0 -0.0035 -0.0150" rpy="0 3.14 0" parent="wrist_yaw_motor" child="AXBrak_Y_R" axis="0 0 1" l="-2" u="+2" v="1.0"/>
+  <xacro:Revjoint id="wrist_yaw" trans="0.04 0 -0.055" rpy="0 -1.57 0" parent="wrist_yaw_motor" child="AXBrak_Y_R" axis="0 0 1" l="-2" u="+2" v="1.0"/>
   <xacro:FxdJoint id="AXBYR_R" trans="0 0 0" parent="AXBrak_Y_R" child="wrist_roll_motor"/>
-  <xacro:Revjoint id="wrist_roll" trans="0 0.0 0.0409163" rpy="0 3.14 0" parent="wrist_roll_motor" child="gripper" axis="0 1 0" l="-2" u="+2" v="1.0"/>
+  <xacro:Revjoint id="wrist_roll" trans="0 0.0 0.0409163" rpy="-1.57 3.14 0" parent="wrist_roll_motor" child="gripper" axis="0 0 1" l="-2" u="+2" v="1.0"/>
   <!--xacro:FxdJoint id="roll_plate_gripper" parent="roll_j_plate" child="gripper" /-->
 </robot>

Commit message: add home in posegoal.py

File: src/mobile_manipulator/model/mobile_manipulator.urdf (robot description, URDF)
Before this commit: robot mobile_manipulator, 15 links, 14 joints
Links:
- link shoulder_yaw_motor: mass 0.140 -> None

File: src/mobile_manipulator/model/mobile_manipulator.xacro (robot description, xacro)
@@ -335,5 +335,5 @@
   </link-->
   <link name="shoulder_yaw_motor">
-    <xacro:MXInertial trans="0 0 0" rpy="0 0 0 "/>
+    <!--xacro:MXInertial trans="0 0 0" rpy="0 0 0 "/-->
     <xacro:MXVisual trans="0 0.188 0.2349" rpy="0 0 0 "/>
     <xacro:MXCollision trans="0 0.188 0.2349" rpy="0 0 0"/>

Commit message: added joint constraints in urdf

File: src/mobile_manipulator/model/mobile_manipulator.urdf (robot description, URDF)
Before this commit: robot mobile_manipulator, 15 links, 14 joints
Joints:
- joint elbow: limit lower=-1.99 upper=1.971699219 effort=30 velocity=1.0 -> lower=-1.9262 upper=1.934 effort=30 velocity=1.0
- joint shoulder_pitch: limit lower=-1.973232422 upper=1.916503906 effort=30 velocity=1.0 -> lower=-1.6592 upper=1.727 effort=30 velocity=1.0
- joint shoulder_yaw: limit lower=-3.0357 upper=3.24426 effort=30 velocity=1.0 -> lower=-3.14 upper=3.14 effort=30 velocity=1.0
- joint wrist_pitch: limit lower=-2.36344086 upper=2.368556533 effort=30 velocity=1.0 -> lower=-2.29 upper=0.718 effort=30 velocity=1.0
- joint wrist_roll: limit lower=-2 upper=+2 effort=30 velocity=1.0 -> lower=-2.617 upper=+2.617 effort=30 velocity=1.0
- joint wrist_yaw: limit lower=-2 upper=+2 effort=30 velocity=1.0 -> lower=-1.43 upper=+2.11 effort=30 velocity=1.0

File: src/mobile_manipulator/model/mobile_manipulator.xacro (robot description, xacro)
@@ -422,19 +422,19 @@
  <!-- JOINTS -->
   <!--xacro:FxdJoint id="bot_joint" parent="bot" child="shoulder_yaw_motor"/-->
-  <xacro:Revjoint id="shoulder_yaw" trans="0 0.188 0.2577" rpy="0 0 3.14" parent="shoulder_yaw_motor" child="shoulder_bracket" axis="0 0 1" l="-3.0357" u="3.24426" v="1.0"/>
+  <xacro:Revjoint id="shoulder_yaw" trans="0 0.188 0.2577" rpy="0 0 3.14" parent="shoulder_yaw_motor" child="shoulder_bracket" axis="0 0 1" l="-3.14" u="3.14" v="1.0"/>
   <!-- 0 0 0.025 -->
-  <xacro:Revjoint id="shoulder_pitch" trans="0 0 0.035" rpy="0 -1.57 0.0" parent="shoulder_bracket" child="shoulder_pitch_motor" axis="0 0 1" l="-1.973232422" u="1.916503906" v="1.0"/>
+  <xacro:Revjoint id="shoulder_pitch" trans="0 0 0.035" rpy="0 -1.57 0.0" parent="shoulder_bracket" child="shoulder_pitch_motor" axis="0 0 1" l="-1.6592" u="1.727" v="1.0"/>
   <xacro:FxdJoint id="s1_l2" trans="0 0 0" parent="shoulder_pitch_motor" child="biscep"/>
   <xacro:FxdJoint id="l2_l2B" trans="0 0 0" parent="biscep" child="elbow_bracket"/>
-  <xacro:Revjoint id="elbow" trans="${0.052 + (length) + 0.038} 0 0" rpy="0 0 0" parent="elbow_bracket" child="elbow_motor" axis="0 0 1" l="-1.99" u="1.971699219" v="1.0"/>
+  <xacro:Revjoint id="elbow" trans="${0.052 + (length) + 0.038} 0 0" rpy="0 0 0" parent="elbow_bracket" child="elbow_motor" axis="0 0 1" l="-1.9262" u="1.934" v="1.0"/>
   <xacro:FxdJoint id="e_l3" trans="0 0 0" parent="elbow_motor" child="forearm"/>
   <xacro:FxdJoint id="l3_l3B" trans="0 0 0" parent="forearm" child="wrist_bracket"/>
-  <xacro:Revjoint id="wrist_pitch" trans="${length + 0.052 + 0.054} 0 0 " rpy="0 0 0" parent="wrist_bracket" child="wrist_pitch_motor" axis="0 0 1" l="-2.36344086" u="2.368556533" v="1.0"/>
+  <xacro:Revjoint id="wrist_pitch" trans="${length + 0.052 + 0.054} 0 0 " rpy="0 0 0" parent="wrist_bracket" child="wrist_pitch_motor" axis="0 0 1" l="-2.29" u="0.718" v="1.0"/>
   <xacro:FxdJoint id="WP_SQ1" trans="0 0 0" parent="wrist_pitch_motor" child="square_plate_1" />
   <xacro:FxdJoint id="SQ1_AXB2B" trans="0 0 0" parent="square_plate_1" child="AXB2B_SQ_Y" />
   <xacro:FxdJoint id="AXB2B_Y" trans="0 0.07 0.055" parent="AXB2B_SQ_Y" child="wrist_yaw_motor" />
-  <xacro:Revjoint id="wrist_yaw" trans="0.04 0 -0.055" rpy="0 -1.57 0" parent="wrist_yaw_motor" child="AXBrak_Y_R" axis="0 0 1" l="-2" u="+2" v="1.0"/>
+  <xacro:Revjoint id="wrist_yaw" trans="0.04 0 -0.055" rpy="0 -1.57 0" parent="wrist_yaw_motor" child="AXBrak_Y_R" axis="0 0 1" l="-1.43" u="+2.11" v="1.0"/>
   <xacro:FxdJoint id="AXBYR_R" trans="0 0 0" parent="AXBrak_Y_R" child="wrist_roll_motor"/>
-  <xacro:Revjoint id="wrist_roll" trans="0 0.0 0.0409163" rpy="-1.57 3.14 0" parent="wrist_roll_motor" child="gripper" axis="0 0 1" l="-2" u="+2" v="1.0"/>
+  <xacro:Revjoint id="wrist_roll" trans="0 0.0 0.0409163" rpy="-1.57 3.14 0" parent="wrist_roll_motor" child="gripper" axis="0 0 1" l="-2.617" u="+2.617" v="1.0"/>
   <!--xacro:FxdJoint id="roll_plate_gripper" parent="roll_j_plate" child="gripper" /-->
 </robot>

Commit message: add bot and moveit config update

File: src/mobile_manipulator/model/mobile_manipulator.urdf (robot description, URDF)
Before this commit: robot mobile_manipulator, 15 links, 14 joints
Links:
- added link bot, mass 0.140; collision mesh filename=package://mobile_manipulator/meshes/bot.stl scale=0.001 0.001 0.001; visual mesh filename=package://mobile_manipulator/meshes/bot.stl scale=0.001 0.001 0.001
Joints:
- added joint bot_joint: type fixed, parent bot, child shoulder_yaw_motor, origin xyz=0 0 0 rpy=0 0 -1.57
- joint AXB2B_Y: origin xyz=0 0.07 0.055 -> xyz=0 0.07 0.055 rpy=0 0 0
- joint AXBYR_R: origin xyz=0 0 0 -> xyz=0 0 0 rpy=0 0 0
- joint SQ1_AXB2B: origin xyz=0 0 0 -> xyz=0 0 0 rpy=0 0 0
- joint WP_SQ1: origin xyz=0 0 0 -> xyz=0 0 0 rpy=0 0 0
- joint e_l3: origin xyz=0 0 0 -> xyz=0 0 0 rpy=0 0 0
- joint l2_l2B: origin xyz=0 0 0 -> xyz=0 0 0 rpy=0 0 0
- joint l3_l3B: origin xyz=0 0 0 -> xyz=0 0 0 rpy=0 0 0
- joint s1_l2: origin xyz=0 0 0 -> xyz=0 0 0 rpy=0 0 0

File: src/mobile_manipulator/model/mobile_manipulator.xacro (robot description, xacro)
@@ -297,7 +297,7 @@
     </joint>
 </xacro:macro>
-<xacro:macro name="FxdJoint" params="id trans parent child">
+<xacro:macro name="FxdJoint" params="id trans rpy parent child">
     <joint name="${id}" type="fixed">
-      <origin xyz="${trans}"/>
+      <origin xyz="${trans}"  rpy="${rpy}" />
       <parent link="${parent}"/>
       <child link="${child}"/>
@@ -329,9 +329,9 @@
 </xacro:macro>
 <!-- LINKS -->
-  <!--link name="bot">
-    <xacro:BotInertial trans="0 0 0" rpy="0 0 0 "/>
-    <xacro:BotVisual trans="0 0 0" rpy="0 0 0 "/>
-    <xacro:BotCollision trans="0 0 0" rpy="0 0 0"/>
-  </link-->
+  <link name="bot">
+    <xacro:BotInertial trans="0 0 0" rpy="0 0 -1.57"/>
+    <xacro:BotVisual trans="0 0 0" rpy="0 0 -1.57"/>
+    <xacro:BotCollision trans="0 0 0" rpy="0 0 -1.57"/>
+  </link>
   <link name="shoulder_yaw_motor">
     <!--xacro:MXInertial trans="0 0 0" rpy="0 0 0 "/-->
@@ -421,19 +421,19 @@
   <!-- 0.0812 -->
  <!-- JOINTS -->
-  <!--xacro:FxdJoint id="bot_joint" parent="bot" child="shoulder_yaw_motor"/-->
+  <xacro:FxdJoint id="bot_joint" trans="0 0 0" rpy="0 0 -1.57" parent="bot" child="shoulder_yaw_motor"/>
   <xacro:Revjoint id="shoulder_yaw" trans="0 0.188 0.2577" rpy="0 0 3.14" parent="shoulder_yaw_motor" child="shoulder_bracket" axis="0 0 1" l="-3.14" u="3.14" v="1.0"/>
   <!-- 0 0 0.025 -->
   <xacro:Revjoint id="shoulder_pitch" trans="0 0 0.035" rpy="0 -1.57 0.0" parent="shoulder_bracket" child="shoulder_pitch_motor" axis="0 0 1" l="-1.6592" u="1.727" v="1.0"/>
-  <xacro:FxdJoint id="s1_l2" trans="0 0 0" parent="shoulder_pitch_motor" child="biscep"/>
-  <xacro:FxdJoint id="l2_l2B" trans="0 0 0" parent="biscep" child="elbow_bracket"/>
+  <xacro:FxdJoint id="s1_l2" trans="0 0 0" rpy="0 0 0" parent="shoulder_pitch_motor" child="biscep"/>
+  <xacro:FxdJoint id="l2_l2B" trans="0 0 0" rpy="0 0 0" parent="biscep" child="elbow_bracket"/>
   <xacro:Revjoint id="elbow" trans="${0.052 + (length) + 0.038} 0 0" rpy="0 0 0" parent="elbow_bracket" child="elbow_motor" axis="0 0 1" l="-1.9262" u="1.934" v="1.0"/>
-  <xacro:FxdJoint id="e_l3" trans="0 0 0" parent="elbow_motor" child="forearm"/>
-  <xacro:FxdJoint id="l3_l3B" trans="0 0 0" parent="forearm" child="wrist_bracket"/>
+  <xacro:FxdJoint id="e_l3" trans="0 0 0" rpy="0 0 0" parent="elbow_motor" child="forearm"/>
+  <xacro:FxdJoint id="l3_l3B" trans="0 0 0" rpy="0 0 0" parent="forearm" child="wrist_bracket"/>
   <xacro:Revjoint id="wrist_pitch" trans="${length + 0.052 + 0.054} 0 0 " rpy="0 0 0" parent="wrist_bracket" child="wrist_pitch_motor" axis="0 0 1" l="-2.29" u="0.718" v="1.0"/>
-  <xacro:FxdJoint id="WP_SQ1" trans="0 0 0" parent="wrist_pitch_motor" child="square_plate_1" />
-  <xacro:FxdJoint id="SQ1_AXB2B" trans="0 0 0" parent="square_plate_1" child="AXB2B_SQ_Y" />
-  <xacro:FxdJoint id="AXB2B_Y" trans="0 0.07 0.055" parent="AXB2B_SQ_Y" child="wrist_yaw_motor" />
+  <xacro:FxdJoint id="WP_SQ1" trans="0 0 0" rpy="0 0 0" parent="wrist_pitch_motor" child="square_plate_1" />
+  <xacro:FxdJoint id="SQ1_AXB2B" trans="0 0 0" rpy="0 0 0" parent="square_plate_1" child="AXB2B_SQ_Y" />
+  <xacro:FxdJoint id="AXB2B_Y" trans="0 0.07 0.055" rpy="0 0 0" parent="AXB2B_SQ_Y" child="wrist_yaw_motor" />
   <xacro:Revjoint id="wrist_yaw" trans="0.04 0 -0.055" rpy="0 -1.57 0" parent="wrist_yaw_motor" child="AXBrak_Y_R" axis="0 0 1" l="-1.43" u="+2.11" v="1.0"/>
-  <xacro:FxdJoint id="AXBYR_R" trans="0 0 0" parent="AXBrak_Y_R" child="wrist_roll_motor"/>
+  <xacro:FxdJoint id="AXBYR_R" trans="0 0 0" rpy="0 0 0" parent="AXBrak_Y_R" child="wrist_roll_motor"/>
   <xacro:Revjoint id="wrist_roll" trans="0 0.0 0.0409163" rpy="-1.57 3.14 0" parent="wrist_roll_motor" child="gripper" axis="0 0 1" l="-2.617" u="+2.617" v="1.0"/>
   <!--xacro:FxdJoint id="roll_plate_gripper" parent="roll_j_plate" child="gripper" /-->

Commit message: removed inertia warning in urdf

File: src/mobile_manipulator/model/mobile_manipulator.urdf (robot description, URDF)
Before this commit: robot mobile_manipulator, 16 links, 15 joints
Links:
- link bot: mass 0.140 -> None
- link shoulder_yaw_motor: mass None -> 0.140

File: src/mobile_manipulator/model/mobile_manipulator.xacro (robot description, xacro)
@@ -330,10 +330,10 @@
 <!-- LINKS -->
   <link name="bot">
-    <xacro:BotInertial trans="0 0 0" rpy="0 0 -1.57"/>
+    <!--<xacro:BotInertial trans="0 0 0" rpy="0 0 -1.57"/>-->
     <xacro:BotVisual trans="0 0 0" rpy="0 0 -1.57"/>
     <xacro:BotCollision trans="0 0 0" rpy="0 0 -1.57"/>
   </link>
   <link name="shoulder_yaw_motor">
-    <!--xacro:MXInertial trans="0 0 0" rpy="0 0 0 "/-->
+    <xacro:MXInertial trans="0 0 0" rpy="0 0 0 "/>
     <xacro:MXVisual trans="0 0.188 0.2349" rpy="0 0 0 "/>
     <xacro:MXCollision trans="0 0.188 0.2349" rpy="0 0 0"/>
