Commit message: urdf j_plate add

File: src/mobile_manipulator/model/mobile_manipulator.urdf (robot description, URDF)
Before this commit: robot mobile_manipulator, 16 links, 15 joints
Links:
- added link roll_j_plate, mass 0.140; collision mesh filename=package://mobile_manipulator/meshes/gripper_Centering.stl scale=0.001 0.001 0.001; visual mesh filename=package://mobile_manipulator/meshes/gripper_Centering.stl scale=0.001 0.001 0.001
Joints:
- added joint roll_plate_gripper: type fixed, parent roll_j_plate, child gripper, origin xyz=-0.0178 -0.043385 0.0025 rpy=0 0 0
- joint wrist_roll: child gripper -> roll_j_plate; origin xyz=0 0.0 0.0409163 rpy=-1.57 3.14 0 -> xyz=0 0 0.0409163 rpy=-1.57 3.14 0

File: src/mobile_manipulator/model/mobile_manipulator.xacro (robot description, xacro)
@@ -389,9 +389,9 @@
     <xacro:AXCollision trans="0 0.002565 0.04237" rpy="-1.57 3.14 0"/>
   </link>
- <!--link name="roll_j_plate">
-    <xacro:roll_j_plate_Inertial trans="0.015 0.0147 0.058" rpy="3.14 1.57 -1.57"/>
-    <xacro:roll_j_plate_Visual trans="0.015 0.0147 0.058" rpy="3.14 1.57 -1.57"/>
-    <xacro:roll_j_plate_Collision trans="0.015 0.0147 0.058" rpy="3.14 1.57 -1.57"/>
-  </link-->
+ <link name="roll_j_plate">
+    <xacro:roll_j_plate_Inertial trans="0.0208 -0.051385 0.0204234" rpy="0 0 1.57"/>
+    <xacro:roll_j_plate_Visual trans="0.0208 -0.051385 0.0204234" rpy="0 0 1.57"/>
+    <xacro:roll_j_plate_Collision trans="0.0208  -0.051385 0.0204234" rpy="0 0 1.57"/>
+  </link>
   <link name="square_plate_1">
     <xacro:square_plate_Inertial trans="0.035 -0.0156 0.02" rpy="-1.57 0 0"/>
@@ -436,5 +436,5 @@
   <xacro:Revjoint id="wrist_yaw" trans="0.04 0 -0.055" rpy="0 -1.57 0" parent="wrist_yaw_motor" child="AXBrak_Y_R" axis="0 0 1" l="-1.43" u="+2.11" v="1.0"/>
   <xacro:FxdJoint id="AXBYR_R" trans="0 0 0" rpy="0 0 0" parent="AXBrak_Y_R" child="wrist_roll_motor"/>
-  <xacro:Revjoint id="wrist_roll" trans="0 0.0 0.0409163" rpy="-1.57 3.14 0" parent="wrist_roll_motor" child="gripper" axis="0 0 1" l="-2.617" u="+2.617" v="1.0"/>
-  <!--xacro:FxdJoint id="roll_plate_gripper" parent="roll_j_plate" child="gripper" /-->
+  <xacro:Revjoint id="wrist_roll" trans="0 0 0.0409163" rpy="-1.57 3.14 0" parent="wrist_roll_motor" child="roll_j_plate" axis="0 0 1" l="-2.617" u="+2.617" v="1.0"/>
+ <xacro:FxdJoint id="roll_plate_gripper" trans="-0.0178 -0.043385 0.0025" rpy="0 0 0" parent="roll_j_plate" child="gripper" />
 </robot>

Commit message: remove fixed joint from urdf

File: src/mobile_manipulator/model/mobile_manipulator.urdf (robot description, URDF)
Before this commit: robot mobile_manipulator, 17 links, 16 joints
Links:
- removed link AXB2B_SQ_Y
- removed link AXBrak_Y_R
- removed link biscep
- removed link elbow_bracket
- removed link forearm
- removed link gripper
- removed link roll_j_plate
- removed link square_plate_1
- removed link wrist_bracket
- link elbow_motor: geometry collision mesh filename=package://mobile_manipulator/meshes/elbow_pitch.STL scale=0.001 0.001 0.001; visual mesh filename=package://mobile_manipulator/meshes/elbow_pitch.STL scale=0.001 0.001 0.001
- link shoulder_bracket: mass 0.00712 -> 0.140; geometry collision mesh filename=package://mobile_manipulator/meshes/shoulder_yaw1.STL scale=0.001 0.001 0.001; visual mesh filename=package://mobile_manipulator/meshes/shoulder_yaw1.STL scale=0.001 0.001 0.001
- link shoulder_pitch_motor: geometry collision mesh filename=package://mobile_manipulator/meshes/shoulder_pitch.STL scale=0.001 0.001 0.001; visual mesh filename=package://mobile_manipulator/meshes/shoulder_pitch.STL scale=0.001 0.001 0.001
- link shoulder_yaw_motor: geometry collision mesh filename=package://mobile_manipulator/meshes/shoulder_yaw.STL scale=0.001 0.001 0.001; visual mesh filename=package://mobile_manipulator/meshes/base_motor.STL scale=0.001 0.001 0.001
- link wrist_pitch_motor: mass 0.05573 -> 0.140; geometry collision mesh filename=package://mobile_manipulator/meshes/wrist_pitch.STL scale=0.001 0.001 0.001; visual mesh filename=package://mobile_manipulator/meshes/wrist_pitch.STL scale=0.001 0.001 0.001
- link wrist_roll_motor: mass 0.05573 -> 0.140; geometry collision mesh filename=package://mobile_manipulator/meshes/wrist_roll.STL scale=0.001 0.001 0.001; visual mesh filename=package://mobile_manipulator/meshes/wrist_roll.STL scale=0.001 0.001 0.001
- link wrist_yaw_motor: mass 0.05573 -> 0.140; geometry collision mesh filename=package://mobile_manipulator/meshes/wrist_yaw.STL scale=0.001 0.001 0.001; visual mesh filename=package://mobile_manipulator/meshes/wrist_yaw.STL scale=0.001 0.001 0.001
Joints:
- removed joint AXB2B_Y
- removed joint AXBYR_R
- removed joint SQ1_AXB2B
- removed joint WP_SQ1
- removed joint e_l3
- removed joint l2_l2B
- removed joint l3_l3B
- removed joint roll_plate_gripper
- removed joint s1_l2
- joint bot_joint: origin xyz=0 0 0 rpy=0 0 -1.57 -> xyz=0 0 0 rpy=0 0 0
- joint elbow: axis 0 0 1 -> 0 1 0; origin xyz=0.186 0 0 rpy=0 0 0 -> xyz=-0.002 0 0.2 rpy=0 0 0; parent elbow_bracket -> shoulder_pitch_motor
- joint shoulder_pitch: axis 0 0 1 -> 0 1 0; origin xyz=0 0 0.035 rpy=0 -1.57 0.0 -> xyz=0 0.010 0.040 rpy=0 0 0.0
- joint shoulder_yaw: origin xyz=0 0.188 0.2577 rpy=0 0 3.14 -> xyz=0.1765 -0.003 0.26 rpy=0 0 0
- joint wrist_pitch: axis 0 0 1 -> 0 1 0; origin xyz=0.202 0 0  rpy=0 0 0 -> xyz=0.004 0 0.196  rpy=0 0 0; parent wrist_bracket -> elbow_motor
- joint wrist_roll: axis 0 0 1 -> 1 0 0; child roll_j_plate -> wrist_roll_motor; origin xyz=0 0 0.0409163 rpy=-1.57 3.14 0 -> xyz=0 0 -0.0415 rpy=0 0 0; parent wrist_roll_motor -> wrist_yaw_motor
- joint wrist_yaw: child AXBrak_Y_R -> wrist_yaw_motor; origin xyz=0.04 0 -0.055 rpy=0 -1.57 0 -> xyz=-0.080 0 0.05 rpy=0 0 0; parent wrist_yaw_motor -> wrist_pitch_motor

File: src/mobile_manipulator/model/mobile_manipulator.xacro (robot description, xacro)
@@ -1,6 +1,12 @@
 <?xml version ="1.0"?>
 <robot xmlns:xacro="http://www.ros.org/wiki/xacro" name="mobile_manipulator">
+<material name="orange">
+  <color rgba="1 0.487 0 1"/>
+</material>
 <material name="white">
   <color rgba="1 1 1 1"/>
+</material>
+<material name="green">
+  <color rgba="0 0.8 0 1"/>
 </material>
 <xacro:property name="MXLength" value="0.0611"/>
@@ -11,290 +17,6 @@
 <xacro:property name="AXDepth" value="0.04"/>
 <xacro:property name="length" value="0.096"/>
-<!-- MACROS -->
-<xacro:macro name="MXInertial" params="trans rpy">
-  <inertial>
-    <origin xyz="${trans}" rpy="${rpy}" />
-    <mass value="0.140" />
-    <inertia ixx="0.000050799110" ixy="0.0" ixz="0.0" iyy="0.00002857215" iyz="0.00000051457" izz="0.000043394" />
-  </inertial>
-</xacro:macro>
-<xacro:macro name="MXVisual" params="trans rpy">
-  <visual>
-    <origin xyz="${trans}" rpy="${rpy}"/>
-    <geometry>
-      <mesh filename="package://mobile_manipulator/meshes/dynamixel_x64series.stl" scale="0.001 0.001 0.001"/>
-    </geometry>
-    <material name="white"/>
-  </visual>
-</xacro:macro>
-<xacro:macro name="MXCollision" params="trans rpy">
-    <collision>
-      <origin xyz="${trans}" rpy="${rpy}"/>
-      <geometry>
-        <box size="0.041 0.0402 0.0611"/>
-      </geometry>
-    </collision>
-</xacro:macro>
-<xacro:macro name="BotInertial" params="trans rpy">
-  <inertial>
-    <origin xyz="${trans}" rpy="${rpy}" />
-    <mass value="0.140" />
-    <inertia ixx="0.000050799110" ixy="0.0" ixz="0.0" iyy="0.00002857215" iyz="0.00000051457" izz="0.000043394" />
-  </inertial>
-</xacro:macro>
-<xacro:macro name="BotVisual" params="trans rpy">
-  <visual>
-    <origin xyz="${trans}" rpy="${rpy}"/>
-    <geometry>
-      <mesh filename="package://mobile_manipulator/meshes/bot.stl" scale="0.001 0.001 0.001"/>
-    </geometry>
-    <material name="white"/>
-  </visual>
-</xacro:macro>
-<xacro:macro name="BotCollision" params="trans rpy">
-    <collision>
-      <origin xyz="${trans}" rpy="${rpy}"/>
-      <geometry>
-        <mesh filename="package://mobile_manipulator/meshes/bot.stl" scale="0.001 0.001 0.001"/>
-      </geometry>
-    </collision>
-</xacro:macro>
-<xacro:macro name="MXCollision_dual_motor" params="trans rpy">
-    <collision>
-      <origin xyz="${trans}" rpy="${rpy}"/>
-      <geometry>
-        <box size="0.041 0.0602 0.1480"/>
-      </geometry>
-    </collision>
-</xacro:macro>
-<xacro:macro name="AXInertial" params="trans rpy">
-  <inertial>
-    <origin xyz="${trans}" rpy="${rpy}"/>
-    <mass value="0.05573" />
-    <inertia ixx="0.00001611154" ixy="0.00000001397" ixz="0.0" iyy="0.00000888743" iyz="0.00000015948" izz="0.00001354172" />
-  </inertial>
-</xacro:macro>
-<xacro:macro name="AXVisual" params="trans rpy">
-  <visual>
-    <origin xyz="${trans}" rpy="${rpy}"/>
-    <geometry>
-      <mesh filename="package://mobile_manipulator/meshes/AX-12_18A - dynamixel_AXseries-1.stl" scale="0.001 0.001 0.001"/>
-    </geometry>
-    <material name="white"/>
-  </visual>
-</xacro:macro>
-<xacro:macro name="AXCollision" params="trans rpy">
-    <collision>
-      <origin xyz="${trans}" rpy="${rpy}"/>
-      <geometry>
-        <box size="0.032 0.04 0.05"/>
-      </geometry>
-    </collision>
-</xacro:macro>
-<xacro:macro name="BracketInertial" params="trans rpy">
-  <inertial>
-    <origin xyz="${trans}" rpy="${rpy}"/>
-    <mass value="0.00712" />
-    <inertia ixx="0.00000174511" iyy="0.00000379922" ixz="0.0" ixy="0.0" iyz="0.0" izz="0.00000357521" />
-  </inertial>
-</xacro:macro>
-<xacro:macro name="BracketVisual" params="trans rpy">
-  <visual>
-    <origin xyz="${trans}" rpy="${rpy}"/>
-    <geometry>
-      <mesh filename="package://mobile_manipulator/meshes/FR05-H101K.stl" scale="0.001 0.001 0.001" />
-    </geometry>
-    <material name="white"/>
-  </visual>
-</xacro:macro>
-<xacro:macro name="BracketCollision" params="trans rpy">
-    <collision>
-      <origin xyz="${trans}" rpy="${rpy}"/>
-      <geometry>
-        <mesh filename="package://mobile_manipulator/meshes/FR05-H101K.stl" scale="0.001 0.001 0.001"/>
-      </geometry>
-    </collision>
-</xacro:macro>
-<xacro:macro name="AxBracketInertial" params="trans rpy">
-  <inertial>
-    <origin xyz="${trans}" rpy="${rpy}"/>
-    <mass value="0.00712" />
-    <inertia ixx="0.00000174511" iyy="0.00000379922" ixz="0.0" ixy="0.0" iyz="0.0" izz="0.00000357521" />
-  </inertial>
-</xacro:macro>
-<xacro:macro name="AxBracketVisual" params="trans rpy">
-  <visual>
-    <origin xyz="${trans}" rpy="${rpy}"/>
-    <geometry>
-      <mesh filename="package://mobile_manipulator/meshes/F4.stl" scale="0.001 0.001 0.001" />
-    </geometry>
-    <material name="white"/>
-  </visual>
-</xacro:macro>
-<xacro:macro name="AxBracketCollision" params="trans rpy">
-    <collision>
-      <origin xyz="${trans}" rpy="${rpy}"/>
-      <geometry>
-        <mesh filename="package://mobile_manipulator/meshes/F4.stl" scale="0.001 0.001 0.001"/>
-      </geometry>
-    </collision>
-</xacro:macro>
-<xacro:macro name="LinkInertial" params="trans rpy">
-  <inertial>
-    <origin xyz="${trans}" rpy="${rpy}"/>
-    <mass value="${0.005*length}" />
-    <inertia ixx="0.000050799110" ixy="0.0" ixz="0.0" iyy="0.00002857215" iyz="0.00000051457" izz="0.000043394"/>
-  </inertial>
-</xacro:macro>
-<xacro:macro name="LinkVisual" params="trans rpy">
-  <visual>
-    <origin xyz="${trans}" rpy="${rpy}"/>
-    <geometry>
-      <box size="0.04 0.04 ${length}"/>
-    </geometry>
-    <material name="white"/>
-  </visual>
-</xacro:macro>
-<xacro:macro name="LinkCollision" params="trans rpy">
-    <collision>
-      <origin xyz="${trans}" rpy="${rpy}"/>
-      <geometry>
-        <box size="0.04 0.04 ${length}"/>
-      </geometry>
-    </collision>
-</xacro:macro>
-<!-- Macros of the J plate -->
-<xacro:macro name="roll_j_plate_Inertial" params="trans rpy">
-  <inertial>
-    <origin xyz="${trans}" rpy="${rpy}" />
-    <mass value="0.140" />
-    <inertia ixx="0.000050799110" ixy="0.0" ixz="0.0" iyy="0.00002857215" iyz="0.00000051457" izz="0.000043394" />
-  </inertial>
-</xacro:macro>
-<xacro:macro name="roll_j_plate_Visual" params="trans rpy">
-  <visual>
-    <origin xyz="${trans}" rpy="${rpy}"/>
-    <geometry>
-      <mesh filename="package://mobile_manipulator/meshes/gripper_Centering.stl" scale="0.001 0.001 0.001"/>
-    </geometry>
-    <material name="white"/>
-  </visual>
-</xacro:macro>
-<xacro:macro name="roll_j_plate_Collision" params="trans rpy">
-    <collision>
-      <origin xyz="${trans}" rpy="${rpy}"/>
-      <geometry>
-        <mesh filename="package://mobile_manipulator/meshes/gripper_Centering.stl" scale="0.001 0.001 0.001"/>
-      </geometry>
-    </collision>
-</xacro:macro>
-<!-- Macros of the square plate -->
-<xacro:macro name="square_plate_Inertial" params="trans rpy">
-  <inertial>
-    <origin xyz="${trans}" rpy="${rpy}" />
-    <mass value="0.140" />
-    <inertia ixx="0.000050799110" ixy="0.0" ixz="0.0" iyy="0.00002857215" iyz="0.00000051457" izz="0.000043394" />
-  </inertial>
-</xacro:macro>
-<xacro:macro name="square_plate_Visual" params="trans rpy">
-  <visual>
-    <origin xyz="${trans}" rpy="${rpy}"/>
-    <geometry>
-      <mesh filename="package://mobile_manipulator/meshes/square_plate.stl" scale="0.001 0.001 0.001"/>
-    </geometry>
-    <material name="white"/>
-  </visual>
-</xacro:macro>
-<xacro:macro name="square_plate_Collision" params="trans rpy">
-    <collision>
-      <origin xyz="${trans}" rpy="${rpy}"/>
-      <geometry>
-        <mesh filename="package://mobile_manipulator/meshes/square_plate.stl" scale="0.001 0.001 0.001"/>
-      </geometry>
-    </collision>
-</xacro:macro>
-<!-- Macros of the gripper -->
-<xacro:macro name="gripper_Inertial" params="trans rpy">
-  <inertial>
-    <origin xyz="${trans}" rpy="${rpy}" />
-    <mass value="0.140" />
-    <inertia ixx="0.000050799110" ixy="0.0" ixz="0.0" iyy="0.00002857215" iyz="0.00000051457" izz="0.000043394" />
-  </inertial>
-</xacro:macro>
-<xacro:macro name="gripper_Visual" params="trans rpy">
-  <visual>
-    <origin xyz="${trans}" rpy="${rpy}"/>
-    <geometry>
-      <mesh filename="package://mobile_manipulator/meshes/gripper.stl" scale="0.001 0.001 0.001"/>
-    </geometry>
-    <material name="white"/>
-  </visual>
-</xacro:macro>
-<xacro:macro name="gripper_Collision" params="trans rpy">
-    <collision>
-      <origin xyz="${trans}" rpy="${rpy}"/>
-      <geometry>
-        <mesh filename="package://mobile_manipulator/meshes/gripper.stl" scale="0.001 0.001 0.001"/>
-      </geometry>
-    </collision>
-</xacro:macro>
-<!-- Macros of the AXBracket -->
-<xacro:macro name="AxBracket_Inertial" params="trans rpy">
-  <inertial>
-    <origin xyz="${trans}" rpy="${rpy}" />
-    <mass value="0.140" />
-    <inertia ixx="0.000050799110" ixy="0.0" ixz="0.0" iyy="0.00002857215" iyz="0.00000051457" izz="0.000043394" />
-  </inertial>
-</xacro:macro>
-<xacro:macro name="AxBracket_Visual" params="trans rpy">
-  <visual>
-    <origin xyz="${trans}" rpy="${rpy}"/>
-    <geometry>
-      <mesh filename="package://mobile_manipulator/meshes/axbracket.stl" scale="0.001 0.001 0.001"/>
-    </geometry>
-    <material name="white"/>
-  </visual>
-</xacro:macro>
-<xacro:macro name="AxBracket_Collision" params="trans rpy">
-    <collision>
-      <origin xyz="${trans}" rpy="${rpy}"/>
-      <geometry>
-        <mesh filename="package://mobile_manipulator/meshes/axbracket.stl" scale="0.001 0.001 0.001"/>
-      </geometry>
-    </collision>
-</xacro:macro>
-<xacro:macro name="AxBack_Inertial" params="trans rpy">
-  <inertial>
-    <origin xyz="${trans}" rpy="${rpy}" />
-    <mass value="0.140" />
-    <inertia ixx="0.000050799110" ixy="0.0" ixz="0.0" iyy="0.00002857215" iyz="0.00000051457" izz="0.000043394" />
-  </inertial>
-</xacro:macro>
-<xacro:macro name="AxBack_Visual" params="trans rpy">
-  <visual>
-    <origin xyz="${trans}" rpy="${rpy}"/>
-    <geometry>
-      <mesh filename="package://mobile_manipulator/meshes/axback.stl" scale="0.001 0.001 0.001"/>
-    </geometry>
-    <material name="white"/>
-  </visual>
-</xacro:macro>
-<xacro:macro name="AxBack_Collision" params="trans rpy">
-    <collision>
-      <origin xyz="${trans}" rpy="${rpy}"/>
-      <geometry>
-        <mesh filename="package://mobile_manipulator/meshes/axback.stl" scale="0.001 0.001 0.001"/>
-      </geometry>
-    </collision>
-</xacro:macro>
-<xacro:macro name="Revjoint" params="id trans rpy parent child axis l u v">
-    <joint name="${id}" type="revolute">
-      <origin xyz="${trans}" rpy="${rpy}"/>
-      <parent link="${parent}"/>
-      <child link="${child}"/>
-      <axis xyz="${axis}"/>
-      <limit lower="${l}" upper="${u}" effort="30" velocity="${v}"/>
-    </joint>
-</xacro:macro>
+============================================================================================================================================
+<!-- FIXED JOINT MACRO-->
 <xacro:macro name="FxdJoint" params="id trans rpy parent child">
     <joint name="${id}" type="fixed">
@@ -304,28 +26,215 @@
     </joint>
 </xacro:macro>
-<xacro:macro name="F10Inertial" params="trans rpy">
-  <inertial>
-    <origin xyz="${trans}" rpy="${rpy}"/>
-    <mass value="0.00712" />
-    <inertia ixx="0.00000174511" iyy="0.00000379922" ixz="0.0" ixy="0.0" iyz="0.0" izz="0.00000357521" />
-  </inertial>
-</xacro:macro>
-<xacro:macro name="F10Visual" params="trans rpy">
-  <visual>
-    <origin xyz="${trans}" rpy="${rpy}"/>
-    <geometry>
-      <mesh filename="package://mobile_manipulator/meshes/F10.stl" scale="0.001 0.001 0.001" />
+<!-- REVOLUTE JOINT MACRO-->
+<xacro:macro name="Revjoint" params="id trans rpy parent child axis l u v">
+    <joint name="${id}" type="revolute">
+      <origin xyz="${trans}" rpy="${rpy}"/>
+      <parent link="${parent}"/>
+      <child link="${child}"/>
+      <axis xyz="${axis}"/>
+      <limit lower="${l}" upper="${u}" effort="30" velocity="${v}"/>
+    </joint>
+</xacro:macro>
+<!-- BOT MACRO-->
+<xacro:macro name="BotInertial" params="trans rpy">
+  <inertial>
+    <origin xyz="${trans}" rpy="${rpy}" />
+    <mass value="0.140" />
+    <inertia ixx="0.000050799110" ixy="0.0" ixz="0.0" iyy="0.00002857215" iyz="0.00000051457" izz="0.000043394" />
+  </inertial>
+</xacro:macro>
+<xacro:macro name="BotVisual" params="trans rpy">
+  <visual>
+    <origin xyz="${trans}" rpy="${rpy}"/>
+    <geometry>
+      <mesh filename="package://mobile_manipulator/meshes/bot.stl" scale="0.001 0.001 0.001"/>
+    </geometry>
+    <material name="green"/>
+  </visual>
+</xacro:macro>
+<xacro:macro name="BotCollision" params="trans rpy">
+    <collision>
+      <origin xyz="${trans}" rpy="${rpy}"/>
+      <geometry>
+        <mesh filename="package://mobile_manipulator/meshes/bot.stl" scale="0.001 0.001 0.001"/>
+      </geometry>
+    </collision>
+</xacro:macro>
+<!-- SHOULDER_YAW MACRO-->
+<xacro:macro name="shoulder_yaw_inertial" params="trans rpy">
+  <inertial>
+    <origin xyz="${trans}" rpy="${rpy}" />
+    <mass value="0.140" />
+    <inertia ixx="0.000050799110" ixy="0.0" ixz="0.0" iyy="0.00002857215" iyz="0.00000051457" izz="0.000043394" />
+  </inertial>
+</xacro:macro>
+<xacro:macro name="shoulder_yaw_visual" params="trans rpy">
+  <visual>
+    <origin xyz="${trans}" rpy="${rpy}"/>
+    <geometry>
+      <mesh filename="package://mobile_manipulator/meshes/base_motor.STL" scale="0.001 0.001 0.001"/>
     </geometry>
     <material name="white"/>
   </visual>
 </xacro:macro>
-<xacro:macro name="F10Collision" params="trans rpy">
-    <collision>
-      <origin xyz="${trans}" rpy="${rpy}"/>
-      <geometry>
-        <mesh filename="package://mobile_manipulator/meshes/F10.stl" scale="0.001 0.001 0.001"/>
-      </geometry>
-    </collision>
-</xacro:macro>
+<xacro:macro name="shoulder_yaw_collision" params="trans rpy">
+    <collision>
+      <origin xyz="${trans}" rpy="${rpy}"/>
+      <geometry>
+        <mesh filename="package://mobile_manipulator/meshes/shoulder_yaw.STL" scale="0.001 0.001 0.001"/>
+      </geometry>
+    </collision>
+</xacro:macro>
+<!-- SHOULDER_BRAK MACRO-->
+<xacro:macro name="shoulder_yaw_brak_inertial" params="trans rpy">
+  <inertial>
+    <origin xyz="${trans}" rpy="${rpy}" />
+    <mass value="0.140" />
+    <inertia ixx="0.000050799110" ixy="0.0" ixz="0.0" iyy="0.00002857215" iyz="0.00000051457" izz="0.000043394" />
+  </inertial>
+</xacro:macro>
+<xacro:macro name="shoulder_yaw_brak_visual" params="trans rpy">
+  <visual>
+    <origin xyz="${trans}" rpy="${rpy}"/>
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