Commit message: 6DOF IKFAST sucessfully done

File: src/mobile_manipulator/model/mobile_manipulator.urdf (robot description, URDF)
Before this commit: robot mobile_manipulator, 8 links, 7 joints
Links:
- link elbow_motor: geometry collision mesh filename=package://mobile_manipulator/meshes/new_elbow_pitch2.STL scale=0.001 0.001 0.001; visual mesh filename=package://mobile_manipulator/meshes/new_elbow_pitch2.STL scale=0.001 0.001 0.001
- link shoulder_bracket: geometry collision mesh filename=package://mobile_manipulator/meshes/shoulder_yaw_brak.STL scale=0.001 0.001 0.001; visual mesh filename=package://mobile_manipulator/meshes/shoulder_yaw_brak.STL scale=0.001 0.001 0.001
- link shoulder_yaw_motor: geometry collision mesh filename=package://mobile_manipulator/meshes/base_motor.STL scale=0.001 0.001 0.001; visual mesh filename=package://mobile_manipulator/meshes/base_motor.STL scale=0.001 0.001 0.001
- link wrist_yaw_motor: geometry collision mesh filename=package://mobile_manipulator/meshes/wrist_yaw_brak.STL scale=0.001 0.001 0.001; visual mesh filename=package://mobile_manipulator/meshes/wrist_yaw_brak.STL scale=0.001 0.001 0.001
Joints:
- joint wrist_pitch: limit lower=-2.29 upper=0.718 effort=30 velocity=1.0 -> lower=-1.43 upper=+2.11 effort=30 velocity=1.0; origin xyz=0.004 0 0.196  rpy=0 0 0 -> xyz=0 0 0 rpy=0 0 0; parent elbow_motor -> wrist_yaw_motor
- joint wrist_roll: origin xyz=0 0 -0.0415 rpy=0 0 0 -> xyz=0 0 0 rpy=0 0 0; parent wrist_yaw_motor -> wrist_pitch_motor
- joint wrist_yaw: limit lower=-1.43 upper=+2.11 effort=30 velocity=1.0 -> lower=-2.29 upper=0.718 effort=30 velocity=1.0; origin xyz=-0.080 0 0.05 rpy=0 0 0 -> xyz=0.015 -0.005 0.278  rpy=0 0 0; parent wrist_pitch_motor -> elbow_motor

File: src/mobile_manipulator/model/mobile_manipulator.xacro (robot description, xacro)
@@ -82,5 +82,5 @@
       <origin xyz="${trans}" rpy="${rpy}"/>
       <geometry>
-        <mesh filename="package://mobile_manipulator/meshes/shoulder_yaw.STL" scale="0.001 0.001 0.001"/>
+        <mesh filename="package://mobile_manipulator/meshes/base_motor.STL" scale="0.001 0.001 0.001"/>
       </geometry>
     </collision>
@@ -98,5 +98,5 @@
     <origin xyz="${trans}" rpy="${rpy}"/>
     <geometry>
-      <mesh filename="package://mobile_manipulator/meshes/shoulder_yaw1.STL" scale="0.001 0.001 0.001"/>
+      <mesh filename="package://mobile_manipulator/meshes/shoulder_yaw_brak.STL" scale="0.001 0.001 0.001"/>
     </geometry>
     <material name="white"/>
@@ -107,5 +107,5 @@
       <origin xyz="${trans}" rpy="${rpy}"/>
       <geometry>
-        <mesh filename="package://mobile_manipulator/meshes/shoulder_yaw1.STL" scale="0.001 0.001 0.001"/>
+        <mesh filename="package://mobile_manipulator/meshes/shoulder_yaw_brak.STL" scale="0.001 0.001 0.001"/>
       </geometry>
     </collision>
@@ -148,5 +148,5 @@
     <origin xyz="${trans}" rpy="${rpy}"/>
     <geometry>
-      <mesh filename="package://mobile_manipulator/meshes/elbow_pitch.STL" scale="0.001 0.001 0.001"/>
+      <mesh filename="package://mobile_manipulator/meshes/new_elbow_pitch2.STL" scale="0.001 0.001 0.001"/>
     </geometry>
     <material name="orange"/>
@@ -157,5 +157,30 @@
       <origin xyz="${trans}" rpy="${rpy}"/>
       <geometry>
-        <mesh filename="package://mobile_manipulator/meshes/elbow_pitch.STL" scale="0.001 0.001 0.001"/>
+        <mesh filename="package://mobile_manipulator/meshes/new_elbow_pitch2.STL" scale="0.001 0.001 0.001"/>
+      </geometry>
+    </collision>
+</xacro:macro>
+<!-- WRIST_YAW_BRAK MACRO-->
+<xacro:macro name="wrist_yaw_inertial" params="trans rpy">
+  <inertial>
+    <origin xyz="${trans}" rpy="${rpy}" />
+    <mass value="0.140" />
+    <inertia ixx="0.000050799110" ixy="0.0" ixz="0.0" iyy="0.00002857215" iyz="0.00000051457" izz="0.000043394" />
+  </inertial>
+</xacro:macro>
+<xacro:macro name="wrist_yaw_visual" params="trans rpy">
+  <visual>
+    <origin xyz="${trans}" rpy="${rpy}"/>
+    <geometry>
+      <mesh filename="package://mobile_manipulator/meshes/wrist_yaw_brak.STL" scale="0.001 0.001 0.001"/>
+    </geometry>
+    <material name="orange"/>
+  </visual>
+</xacro:macro>
+<xacro:macro name="wrist_yaw_collision" params="trans rpy">
+    <collision>
+      <origin xyz="${trans}" rpy="${rpy}"/>
+      <geometry>
+        <mesh filename="package://mobile_manipulator/meshes/wrist_yaw_brak.STL" scale="0.001 0.001 0.001"/>
       </geometry>
     </collision>
@@ -183,29 +208,4 @@
       <geometry>
         <mesh filename="package://mobile_manipulator/meshes/wrist_pitch.STL" scale="0.001 0.001 0.001"/>
-      </geometry>
-    </collision>
-</xacro:macro>
-<!-- WRIST_YAW MACRO-->
-<xacro:macro name="wrist_yaw_inertial" params="trans rpy">
-  <inertial>
-    <origin xyz="${trans}" rpy="${rpy}" />
-    <mass value="0.140" />
-    <inertia ixx="0.000050799110" ixy="0.0" ixz="0.0" iyy="0.00002857215" iyz="0.00000051457" izz="0.000043394" />
-  </inertial>
-</xacro:macro>
-<xacro:macro name="wrist_yaw_visual" params="trans rpy">
-  <visual>
-    <origin xyz="${trans}" rpy="${rpy}"/>
-    <geometry>
-      <mesh filename="package://mobile_manipulator/meshes/wrist_yaw.STL" scale="0.001 0.001 0.001"/>
-    </geometry>
-    <material name="orange"/>
-  </visual>
-</xacro:macro>
-<xacro:macro name="wrist_yaw_collision" params="trans rpy">
-    <collision>
-      <origin xyz="${trans}" rpy="${rpy}"/>
-      <geometry>
-        <mesh filename="package://mobile_manipulator/meshes/wrist_yaw.STL" scale="0.001 0.001 0.001"/>
       </geometry>
     </collision>
@@ -259,22 +259,22 @@
   </link>
   <link name="elbow_motor">
-    <xacro:elbow_inertial trans="0.0180 -0.09 -0.02" rpy="-1.57 3.14 0"/>
-    <xacro:elbow_visual trans="0.0180 -0.09 -0.02" rpy="-1.57 3.14 0"/>
-    <xacro:elbow_collision trans="0.0180 -0.09 -0.02" rpy="-1.57 3.14 0"/>
+    <xacro:elbow_inertial trans="-0.025 0.075 -0.02" rpy="-1.57 3.14 3.14"/>
+    <xacro:elbow_visual trans="-0.025  0.085 -0.02" rpy="-1.57 3.14 3.14"/>
+    <xacro:elbow_collision trans="-0.025 0.075 -0.02" rpy="-1.57 3.14 3.14"/>
+  </link>
+  <link name="wrist_yaw_motor">
+    <xacro:wrist_yaw_inertial trans="0.0 0 -0.052" rpy="0 0 0"/>
+    <xacro:wrist_yaw_visual trans="-0.025 0.048 -0.052" rpy="1.57 0 0"/>
+    <xacro:wrist_yaw_collision trans="0.0 0 -0.052" rpy="0 0 0"/>
   </link>
   <link name="wrist_pitch_motor">
-    <xacro:wrist_pitch_inertial trans="0.0090 -0.05 -0.009" rpy="-1.57 0 1.57"/>
-    <xacro:wrist_pitch_visual trans="0.0090 -0.05 -0.009" rpy="-1.57 3.14 0"/>
-    <xacro:wrist_pitch_collision trans="0.0090 -0.05 -0.009" rpy="-1.57 0 1.57"/>
-  </link>
-  <link name="wrist_yaw_motor">
-    <xacro:wrist_yaw_inertial trans="0.02 -0.055 -0.063" rpy="0 0 3.14"/>
-    <xacro:wrist_yaw_visual trans="0.02 -0.055 -0.063" rpy="1.57 0 3.14"/>
-    <xacro:wrist_yaw_collision trans="0.02 -0.055 -0.063" rpy="0 0 3.14"/>
+    <xacro:wrist_pitch_inertial trans="0.0 0.051 -0.009" rpy="-1.57 0 1.57"/>
+    <xacro:wrist_pitch_visual trans="-0.0165 0.051 -0.008" rpy="-1.57 3.14 3.14"/>
+    <xacro:wrist_pitch_collision trans="0.0 0.051 -0.009" rpy="-1.57 0 1.57"/>
   </link>
   <link name="wrist_roll_motor">
-    <xacro:wrist_roll_inertial trans="-0.02 -0.06 -0.026" rpy="-1.57 3.14 0"/>
-    <xacro:wrist_roll_visual trans="-0.02 -0.06 -0.026" rpy="-1.57 3.14 0"/>
-    <xacro:wrist_roll_collision trans="-0.02 -0.06 -0.026" rpy="-1.57 3.14 0"/>
+    <xacro:wrist_roll_inertial trans="-0.02 -0.06 -0.026" rpy="-1.57 3.14 3.14"/>
+    <xacro:wrist_roll_visual trans="0.057 0.05 -0.015" rpy="-1.57 3.14 3.14"/>
+    <xacro:wrist_roll_collision trans="-0.02 -0.06 -0.026" rpy="-1.57 3.14 3.14"/>
   </link>
  <!-- JOINTS -->
@@ -283,6 +283,6 @@
   <xacro:Revjoint id="shoulder_pitch" trans="0 0.010 0.040" rpy="0 0 0.0" parent="shoulder_bracket" child="shoulder_pitch_motor" axis="0 1 0" l="-1.6592" u="1.727" v="1.0"/>
   <xacro:Revjoint id="elbow" trans="${0.052 + (length) - 0.150} 0 0.2" rpy="0 0 0" parent="shoulder_pitch_motor" child="elbow_motor" axis="0 1 0" l="-1.9262" u="1.934" v="1.0"/>
-  <xacro:Revjoint id="wrist_pitch" trans="${length + 0.052 - 0.144} 0 0.196 " rpy="0 0 0" parent="elbow_motor" child="wrist_pitch_motor" axis="0 1 0" l="-2.29" u="0.718" v="1.0"/>
-  <xacro:Revjoint id="wrist_yaw" trans="-0.080 0 0.05" rpy="0 0 0" parent="wrist_pitch_motor" child="wrist_yaw_motor" axis="0 0 1" l="-1.43" u="+2.11" v="1.0"/>
-  <xacro:Revjoint id="wrist_roll" trans="0 0 -0.0415" rpy="0 0 0" parent="wrist_yaw_motor" child="wrist_roll_motor" axis="1 0 0" l="-2.617" u="+2.617" v="1.0"/>
+  <xacro:Revjoint id="wrist_yaw" trans="0.015 -0.005 0.278 " rpy="0 0 0" parent="elbow_motor" child="wrist_yaw_motor" axis="0 0 1" l="-2.29" u="0.718" v="1.0"/>
+  <xacro:Revjoint id="wrist_pitch" trans="0 0 0" rpy="0 0 0" parent="wrist_yaw_motor" child="wrist_pitch_motor" axis="0 1 0" l="-1.43" u="+2.11" v="1.0"/>
+  <xacro:Revjoint id="wrist_roll" trans="0 0 0" rpy="0 0 0" parent="wrist_pitch_motor" child="wrist_roll_motor" axis="1 0 0" l="-2.617" u="+2.617" v="1.0"/>
 </robot>

Commit message: change limits in xacro

File: src/mobile_manipulator/model/mobile_manipulator.urdf (robot description, URDF)
Before this commit: robot mobile_manipulator, 8 links, 7 joints
Joints:
- joint elbow: limit lower=-1.9262 upper=1.934 effort=30 velocity=1.0 -> lower=-1.9880391011 upper=1.97730123558 effort=30 velocity=1.0
- joint shoulder_pitch: limit lower=-1.6592 upper=1.727 effort=30 velocity=1.0 -> lower=-1.59 upper=1.97423327401 effort=30 velocity=1.0
- joint wrist_pitch: limit lower=-1.43 upper=+2.11 effort=30 velocity=1.0 -> lower=-2.617 upper=0.99 effort=30 velocity=1.0
- joint wrist_roll: limit lower=-2.617 upper=+2.617 effort=30 velocity=1.0 -> lower=-2.617 upper=2.617 effort=30 velocity=1.0
- joint wrist_yaw: limit lower=-2.29 upper=0.718 effort=30 velocity=1.0 -> lower=-2.617 upper=2.617 effort=30 velocity=1.0

File: src/mobile_manipulator/model/mobile_manipulator.xacro (robot description, xacro)
@@ -279,10 +279,10 @@
   </link>
  <!-- JOINTS -->
-  <xacro:FxdJoint id="bot_joint" trans="0 0 0" rpy="0 0 0" parent="bot" child="shoulder_yaw_motor"/>
+   <xacro:FxdJoint id="bot_joint" trans="0 0 0" rpy="0 0 0" parent="bot" child="shoulder_yaw_motor"/>
   <xacro:Revjoint id="shoulder_yaw" trans="0.1765 -0.003 0.26" rpy="0 0 0" parent="shoulder_yaw_motor" child="shoulder_bracket" axis="0 0 1" l="-3.14" u="3.14" v="1.0"/>
-  <xacro:Revjoint id="shoulder_pitch" trans="0 0.010 0.040" rpy="0 0 0.0" parent="shoulder_bracket" child="shoulder_pitch_motor" axis="0 1 0" l="-1.6592" u="1.727" v="1.0"/>
-  <xacro:Revjoint id="elbow" trans="${0.052 + (length) - 0.150} 0 0.2" rpy="0 0 0" parent="shoulder_pitch_motor" child="elbow_motor" axis="0 1 0" l="-1.9262" u="1.934" v="1.0"/>
-  <xacro:Revjoint id="wrist_yaw" trans="0.015 -0.005 0.278 " rpy="0 0 0" parent="elbow_motor" child="wrist_yaw_motor" axis="0 0 1" l="-2.29" u="0.718" v="1.0"/>
-  <xacro:Revjoint id="wrist_pitch" trans="0 0 0" rpy="0 0 0" parent="wrist_yaw_motor" child="wrist_pitch_motor" axis="0 1 0" l="-1.43" u="+2.11" v="1.0"/>
-  <xacro:Revjoint id="wrist_roll" trans="0 0 0" rpy="0 0 0" parent="wrist_pitch_motor" child="wrist_roll_motor" axis="1 0 0" l="-2.617" u="+2.617" v="1.0"/>
+  <xacro:Revjoint id="shoulder_pitch" trans="0 0.010 0.040" rpy="0 0 0.0" parent="shoulder_bracket" child="shoulder_pitch_motor" axis="0 1 0" l="-1.59" u="1.97423327401" v="1.0"/>
+  <xacro:Revjoint id="elbow" trans="${0.052 + (length) - 0.150} 0 0.2" rpy="0 0 0" parent="shoulder_pitch_motor" child="elbow_motor" axis="0 1 0" l="-1.9880391011" u="1.97730123558" v="1.0"/>
+  <xacro:Revjoint id="wrist_yaw" trans="0.015 -0.005 0.278 " rpy="0 0 0" parent="elbow_motor" child="wrist_yaw_motor" axis="0 0 1" l="-2.617" u="2.617" v="1.0"/>
+  <xacro:Revjoint id="wrist_pitch" trans="0 0 0" rpy="0 0 0" parent="wrist_yaw_motor" child="wrist_pitch_motor" axis="0 1 0" l="-2.617" u="0.99" v="1.0"/>
+  <xacro:Revjoint id="wrist_roll" trans="0 0 0" rpy="0 0 0" parent="wrist_pitch_motor" child="wrist_roll_motor" axis="1 0 0" l="-2.617" u="2.617" v="1.0"/>
 </robot>

Commit message: seperate gripper

File: src/mobile_manipulator/model/mobile_manipulator.urdf (robot description, URDF)
Before this commit: robot mobile_manipulator, 8 links, 7 joints
Joints:
- joint wrist_yaw: origin xyz=0.015 -0.005 0.278  rpy=0 0 0 -> xyz= 0.015 -0.005 0.278 rpy=0 0 0

File: src/mobile_manipulator/model/mobile_manipulator.xacro (robot description, xacro)
@@ -236,4 +236,29 @@
     </collision>
 </xacro:macro>
+<!-- GRIPPER MACRO-->
+<xacro:macro name="gripper_inertial" params="trans rpy">
+  <inertial>
+    <origin xyz="${trans}" rpy="${rpy}" />
+    <mass value="0.140" />
+    <inertia ixx="0.000050799110" ixy="0.0" ixz="0.0" iyy="0.00002857215" iyz="0.00000051457" izz="0.000043394" />
+  </inertial>
+</xacro:macro>
+<xacro:macro name="gripper_visual" params="trans rpy">
+  <visual>
+    <origin xyz="${trans}" rpy="${rpy}"/>
+    <geometry>
+      <mesh filename="package://mobile_manipulator/meshes/gripper_wheel.STL" scale="0.001 0.001 0.001"/>
+    </geometry>
+    <material name="orange"/>
+  </visual>
+</xacro:macro>
+<xacro:macro name="gripper_collision" params="trans rpy">
+    <collision>
+      <origin xyz="${trans}" rpy="${rpy}"/>
+      <geometry>
+        <mesh filename="package://mobile_manipulator/meshes/gripper_wheel.STL" scale="0.001 0.001 0.001"/>
+      </geometry>
+    </collision>
+</xacro:macro>
 =============================================================================================================================================
 <!-- LINKS -->
@@ -274,7 +299,12 @@
   </link>
   <link name="wrist_roll_motor">
-    <xacro:wrist_roll_inertial trans="0.057 0.05 -0.015" rpy="-1.57 3.14 3.14"/>
-    <xacro:wrist_roll_visual trans="0.057 0.05 -0.015" rpy="-1.57 3.14 3.14"/>
-    <xacro:wrist_roll_collision trans="0.057 0.05 -0.015" rpy="-1.57 3.14 3.14"/>
+    <xacro:wrist_roll_inertial trans="0.057 0.11 -0.01" rpy="-1.57 3.14 3.14"/>
+    <xacro:wrist_roll_visual trans="0.057 0.11 -0.01" rpy="-1.57 3.14 3.14"/>
+    <xacro:wrist_roll_collision trans="0.057 0.11 -0.01" rpy="-1.57 3.14 3.14"/>
+  </link>
+  <link name="gripper_motor">
+  	<xacro:gripper_inertial trans="-0.016 0.016 0 " rpy="-1.57 1.57 3.14"/>
+    <xacro:gripper_visual trans="-0.016 0.016 0" rpy="-1.57 1.57 3.14"/>
+    <xacro:gripper_collision trans="-0.016 0.016 0 " rpy="-1.57 1.57 3.14"/>
   </link>
  <!-- JOINTS -->
@@ -283,6 +313,7 @@
   <xacro:Revjoint id="shoulder_pitch" trans="0 0.010 0.040" rpy="0 0 0.0" parent="shoulder_bracket" child="shoulder_pitch_motor" axis="0 1 0" l="-1.59" u="1.97423327401" v="1.0"/>
   <xacro:Revjoint id="elbow" trans="${0.052 + (length) - 0.150} 0 0.2" rpy="0 0 0" parent="shoulder_pitch_motor" child="elbow_motor" axis="0 1 0" l="-1.9880391011" u="1.97730123558" v="1.0"/>
-  <xacro:Revjoint id="wrist_yaw" trans="0.015 -0.005 0.278 " rpy="0 0 0" parent="elbow_motor" child="wrist_yaw_motor" axis="0 0 1" l="-2.617" u="2.617" v="1.0"/>
+  <xacro:Revjoint id="wrist_yaw" trans=" 0.015 -0.005 0.278" rpy="0 0 0" parent="elbow_motor" child="wrist_yaw_motor" axis="0 0 1" l="-2.617" u="2.617" v="1.0"/>
   <xacro:Revjoint id="wrist_pitch" trans="0 0 0" rpy="0 0 0" parent="wrist_yaw_motor" child="wrist_pitch_motor" axis="0 1 0" l="-2.617" u="0.99" v="1.0"/>
   <xacro:Revjoint id="wrist_roll" trans="0 0 0" rpy="0 0 0" parent="wrist_pitch_motor" child="wrist_roll_motor" axis="1 0 0" l="-2.617" u="2.617" v="1.0"/>
+  <xacro:Revjoint id="gripper" trans="0.1 0.0213 0.024" rpy="0 0 0" parent="wrist_roll_motor" child="gripper_motor" axis="0 0 1" l="-2.617" u="2.617" v="1.0"/>
 </robot>

Commit message: new urdf with gripper joint

File: src/mobile_manipulator/model/mobile_manipulator.urdf (robot description, URDF)
Before this commit: robot mobile_manipulator, 8 links, 7 joints
Links:
- added link gripper_motor, mass 0.140; collision mesh filename=package://mobile_manipulator/meshes/gripper_wheel.STL scale=0.001 0.001 0.001; visual mesh filename=package://mobile_manipulator/meshes/gripper_wheel.STL scale=0.001 0.001 0.001
- link wrist_roll_motor: geometry collision mesh filename=package://mobile_manipulator/meshes/new_wrist_roll.STL scale=0.001 0.001 0.001; visual mesh filename=package://mobile_manipulator/meshes/new_wrist_roll.STL scale=0.001 0.001 0.001
Joints:
- added joint gripper: type revolute, parent wrist_roll_motor, child gripper_motor, origin xyz=0.1 0.0213 0.024 rpy=0 0 0, axis 0 0 1, limit lower=-2.617 upper=2.617 effort=30 velocity=1.0

File: src/mobile_manipulator/model/mobile_manipulator.xacro (robot description, xacro)
@@ -223,5 +223,5 @@
     <origin xyz="${trans}" rpy="${rpy}"/>
     <geometry>
-      <mesh filename="package://mobile_manipulator/meshes/wrist_roll.STL" scale="0.001 0.001 0.001"/>
+      <mesh filename="package://mobile_manipulator/meshes/new_wrist_roll.STL" scale="0.001 0.001 0.001"/>
     </geometry>
     <material name="orange"/>
@@ -232,5 +232,5 @@
       <origin xyz="${trans}" rpy="${rpy}"/>
       <geometry>
-        <mesh filename="package://mobile_manipulator/meshes/wrist_roll.STL" scale="0.001 0.001 0.001"/>
+        <mesh filename="package://mobile_manipulator/meshes/new_wrist_roll.STL" scale="0.001 0.001 0.001"/>
       </geometry>
     </collision>

Commit message: updated urdf with shoulder_yaw_plus

File: src/mobile_manipulator/model/mobile_manipulator.urdf (robot description, URDF)
Before this commit: robot mobile_manipulator, 9 links, 8 joints
Links:
- link shoulder_bracket: geometry collision mesh filename=package://mobile_manipulator/meshes/shoulder_yaw_plus.STL scale=0.001 0.001 0.001; visual mesh filename=package://mobile_manipulator/meshes/shoulder_yaw_plus.STL scale=0.001 0.001 0.001

File: src/mobile_manipulator/model/mobile_manipulator.xacro (robot description, xacro)
@@ -98,5 +98,5 @@
     <origin xyz="${trans}" rpy="${rpy}"/>
     <geometry>
-      <mesh filename="package://mobile_manipulator/meshes/shoulder_yaw_brak.STL" scale="0.001 0.001 0.001"/>
+      <mesh filename="package://mobile_manipulator/meshes/shoulder_yaw_plus.STL" scale="0.001 0.001 0.001"/>
     </geometry>
     <material name="white"/>
@@ -107,5 +107,5 @@
       <origin xyz="${trans}" rpy="${rpy}"/>
       <geometry>
-        <mesh filename="package://mobile_manipulator/meshes/shoulder_yaw_brak.STL" scale="0.001 0.001 0.001"/>
+        <mesh filename="package://mobile_manipulator/meshes/shoulder_yaw_plus.STL" scale="0.001 0.001 0.001"/>
       </geometry>
     </collision>
@@ -274,7 +274,7 @@
   </link>
   <link name="shoulder_bracket">
-    <xacro:shoulder_yaw_brak_inertial trans="-0.019 -0.062 0" rpy="0 0 0 "/>
-    <xacro:shoulder_yaw_brak_visual trans="-0.019 -0.062 0" rpy="0 0 0 "/>
-    <xacro:shoulder_yaw_brak_collision trans="-0.019 -0.062 0" rpy="0 0 0 "/>
+    <xacro:shoulder_yaw_brak_inertial trans="-0.159 -0.095 -0.07" rpy="1.57 0 1.57 "/>
+    <xacro:shoulder_yaw_brak_visual trans="-0.159 -0.095 -0.07" rpy="1.57 0 1.57 "/>
+    <xacro:shoulder_yaw_brak_collision trans="-0.159 -0.095 -0.07" rpy="1.57 0 1.57 "/>
   </link>
   <link name="shoulder_pitch_motor">

Commit message: gripper added to urdf

File: src/mobile_manipulator/model/mobile_manipulator.urdf (robot description, URDF)
Before this commit: robot mobile_manipulator, 9 links, 8 joints
Links:
- link gripper_motor: geometry collision mesh filename=package://mobile_manipulator/meshes/gripper.stl scale=0.001 0.001 0.001; visual mesh filename=package://mobile_manipulator/meshes/gripper.stl scale=0.001 0.001 0.001

File: src/mobile_manipulator/model/mobile_manipulator.xacro (robot description, xacro)
@@ -248,5 +248,5 @@
     <origin xyz="${trans}" rpy="${rpy}"/>
     <geometry>
-      <mesh filename="package://mobile_manipulator/meshes/gripper_wheel.STL" scale="0.001 0.001 0.001"/>
+      <mesh filename="package://mobile_manipulator/meshes/gripper.stl" scale="0.001 0.001 0.001"/>
     </geometry>
     <material name="orange"/>
@@ -257,5 +257,5 @@
       <origin xyz="${trans}" rpy="${rpy}"/>
       <geometry>
-        <mesh filename="package://mobile_manipulator/meshes/gripper_wheel.STL" scale="0.001 0.001 0.001"/>
+        <mesh filename="package://mobile_manipulator/meshes/gripper.stl" scale="0.001 0.001 0.001"/>
       </geometry>
     </collision>
@@ -304,7 +304,7 @@
   </link>
   <link name="gripper_motor">
-  	<xacro:gripper_inertial trans="-0.016 0.016 0 " rpy="-1.57 1.57 3.14"/>
-    <xacro:gripper_visual trans="-0.016 0.016 0" rpy="-1.57 1.57 3.14"/>
-    <xacro:gripper_collision trans="-0.016 0.016 0 " rpy="-1.57 1.57 3.14"/>
+  	<xacro:gripper_inertial trans="0.024 -0.004 -0.05 " rpy="0 0 -1.57"/>
+    <xacro:gripper_visual trans="0.024 -0.004 -0.05" rpy="0 0 -1.57"/>
+    <xacro:gripper_collision trans="0.024 -0.004 -0.05 " rpy="0 0 -1.57"/>
   </link>
  <!-- JOINTS -->
