Commit message: added end_effector cube as link

File: src/mobile_manipulator/model/mobile_manipulator.urdf (robot description, URDF)
Before this commit: robot mobile_manipulator, 9 links, 8 joints
Links:
- removed link gripper_motor
- added link end_effector_link, mass 0.140; collision mesh filename=package://mobile_manipulator/meshes/cube.STL scale=0.001 0.001 0.001; visual mesh filename=package://mobile_manipulator/meshes/cube.STL scale=0.001 0.001 0.001
- link wrist_roll_motor: geometry collision mesh filename=package://mobile_manipulator/meshes/wrist_roll_gripper.STL scale=0.001 0.001 0.001; visual mesh filename=package://mobile_manipulator/meshes/wrist_roll_gripper.STL scale=0.001 0.001 0.001
Joints:
- removed joint gripper
- added joint end_eff_joint: type fixed, parent wrist_roll_motor, child end_effector_link, origin xyz=0.20 0 0.02 rpy=0 0 0

File: src/mobile_manipulator/model/mobile_manipulator.xacro (robot description, xacro)
@@ -223,5 +223,5 @@
     <origin xyz="${trans}" rpy="${rpy}"/>
     <geometry>
-      <mesh filename="package://mobile_manipulator/meshes/new_wrist_roll.STL" scale="0.001 0.001 0.001"/>
+      <mesh filename="package://mobile_manipulator/meshes/wrist_roll_gripper.STL" scale="0.001 0.001 0.001"/>
     </geometry>
     <material name="orange"/>
@@ -232,10 +232,10 @@
       <origin xyz="${trans}" rpy="${rpy}"/>
       <geometry>
-        <mesh filename="package://mobile_manipulator/meshes/new_wrist_roll.STL" scale="0.001 0.001 0.001"/>
+        <mesh filename="package://mobile_manipulator/meshes/wrist_roll_gripper.STL" scale="0.001 0.001 0.001"/>
       </geometry>
     </collision>
 </xacro:macro>
 <!-- GRIPPER MACRO-->
-<xacro:macro name="gripper_inertial" params="trans rpy">
+<!-- <xacro:macro name="gripper_inertial" params="trans rpy">
   <inertial>
     <origin xyz="${trans}" rpy="${rpy}" />
@@ -258,4 +258,28 @@
       <geometry>
         <mesh filename="package://mobile_manipulator/meshes/gripper.stl" scale="0.001 0.001 0.001"/>
+      </geometry>
+    </collision>
+</xacro:macro> -->
+<xacro:macro name="end_eff_inertial" params="trans rpy">
+  <inertial>
+    <origin xyz="${trans}" rpy="${rpy}" />
+    <mass value="0.140" />
+    <inertia ixx="0.000050799110" ixy="0.0" ixz="0.0" iyy="0.00002857215" iyz="0.00000051457" izz="0.000043394" />
+  </inertial>
+</xacro:macro>
+<xacro:macro name="end_eff_visual" params="trans rpy">
+  <visual>
+    <origin xyz="${trans}" rpy="${rpy}"/>
+    <geometry>
+      <mesh filename="package://mobile_manipulator/meshes/cube.STL" scale="0.001 0.001 0.001"/>
+    </geometry>
+    <material name="green"/>
+  </visual>
+</xacro:macro>
+<xacro:macro name="end_eff_collision" params="trans rpy">
+    <collision>
+      <origin xyz="${trans}" rpy="${rpy}"/>
+      <geometry>
+        <mesh filename="package://mobile_manipulator/meshes/cube.STL" scale="0.001 0.001 0.001"/>
       </geometry>
     </collision>
@@ -299,12 +323,12 @@
   </link>
   <link name="wrist_roll_motor">
-    <xacro:wrist_roll_inertial trans="0.057 0.11 -0.01" rpy="-1.57 3.14 3.14"/>
-    <xacro:wrist_roll_visual trans="0.057 0.11 -0.01" rpy="-1.57 3.14 3.14"/>
-    <xacro:wrist_roll_collision trans="0.057 0.11 -0.01" rpy="-1.57 3.14 3.14"/>
-  </link>
-  <link name="gripper_motor">
-  	<xacro:gripper_inertial trans="0.024 -0.004 -0.05 " rpy="0 0 -1.57"/>
-    <xacro:gripper_visual trans="0.024 -0.004 -0.05" rpy="0 0 -1.57"/>
-    <xacro:gripper_collision trans="0.024 -0.004 -0.05 " rpy="0 0 -1.57"/>
+    <xacro:wrist_roll_inertial trans="0.057 0.055 -0.01" rpy="-1.57 3.14 3.14"/>
+    <xacro:wrist_roll_visual trans="0.057 0.055 -0.01" rpy="-1.57 3.14 3.14"/>
+    <xacro:wrist_roll_collision trans="0.057 0.055 -0.01" rpy="-1.57 3.14 3.14"/>
+  </link>
+ <link name="end_effector_link">
+    <xacro:end_eff_inertial trans="-0.04 0 0.005" rpy="-1.57 3.14 3.14"/>
+    <xacro:end_eff_visual trans="-0.04 0 0.005" rpy="-1.57 3.14 3.14"/>
+    <xacro:end_eff_collision trans="-0.04 0 0.005" rpy="-1.57 3.14 3.14"/>
   </link>
  <!-- JOINTS -->
@@ -316,4 +340,4 @@
   <xacro:Revjoint id="wrist_pitch" trans="0 0 0" rpy="0 0 0" parent="wrist_yaw_motor" child="wrist_pitch_motor" axis="0 1 0" l="-2.617" u="0.99" v="1.0"/>
   <xacro:Revjoint id="wrist_roll" trans="0 0 0" rpy="0 0 0" parent="wrist_pitch_motor" child="wrist_roll_motor" axis="1 0 0" l="-2.617" u="2.617" v="1.0"/>
-  <xacro:Revjoint id="gripper" trans="0.1 0.0213 0.024" rpy="0 0 0" parent="wrist_roll_motor" child="gripper_motor" axis="0 0 1" l="-2.617" u="2.617" v="1.0"/>
+  <xacro:FxdJoint id="end_eff_joint" trans="0.20 0 0.02" rpy="0 0 0" parent="wrist_roll_motor" child="end_effector_link"/>
 </robot>

Commit message: Updated urdf according to final bot

File: src/mobile_manipulator/model/mobile_manipulator.urdf (robot description, URDF)
Before this commit: robot mobile_manipulator, 9 links, 8 joints
Joints:
- joint shoulder_pitch: origin xyz=0 0.010 0.040 rpy=0 0 0.0 -> xyz=0.0 0.010 0.040 rpy=0 0 0.0
- joint shoulder_yaw: origin xyz=0.1765 -0.003 0.26 rpy=0 0 0 -> xyz=0.0965 -0.003 0.26 rpy=0 0 0

File: src/mobile_manipulator/model/mobile_manipulator.xacro (robot description, xacro)
@@ -293,7 +293,7 @@
   </link>
   <link name="shoulder_yaw_motor">
-    <xacro:shoulder_yaw_inertial trans="0.13 -0.02 0.1715" rpy="0 0 0 "/>
-    <xacro:shoulder_yaw_visual trans="0.13 -0.02 0.1715" rpy="0 0 0 "/>
-    <xacro:shoulder_yaw_collision trans="0.13 -0.02 0.1715" rpy="0 0 0"/>
+    <xacro:shoulder_yaw_inertial trans="0.05 -0.02 0.1715" rpy="0 0 0 "/>
+    <xacro:shoulder_yaw_visual trans="0.05 -0.02 0.1715" rpy="0 0 0 "/>
+    <xacro:shoulder_yaw_collision trans="0.05 -0.02 0.1715" rpy="0 0 0"/>
   </link>
   <link name="shoulder_bracket">
@@ -334,6 +334,6 @@
  <!-- JOINTS -->
    <xacro:FxdJoint id="bot_joint" trans="0 0 0" rpy="0 0 0" parent="bot" child="shoulder_yaw_motor"/>
-  <xacro:Revjoint id="shoulder_yaw" trans="0.1765 -0.003 0.26" rpy="0 0 0" parent="shoulder_yaw_motor" child="shoulder_bracket" axis="0 0 1" l="-3.14" u="3.14" v="1.0"/>
-  <xacro:Revjoint id="shoulder_pitch" trans="0 0.010 0.040" rpy="0 0 0.0" parent="shoulder_bracket" child="shoulder_pitch_motor" axis="0 1 0" l="-1.59" u="1.97423327401" v="1.0"/>
+  <xacro:Revjoint id="shoulder_yaw" trans="0.0965 -0.003 0.26" rpy="0 0 0" parent="shoulder_yaw_motor" child="shoulder_bracket" axis="0 0 1" l="-3.14" u="3.14" v="1.0"/>
+  <xacro:Revjoint id="shoulder_pitch" trans="0.0 0.010 0.040" rpy="0 0 0.0" parent="shoulder_bracket" child="shoulder_pitch_motor" axis="0 1 0" l="-1.59" u="1.97423327401" v="1.0"/>
   <xacro:Revjoint id="elbow" trans="${0.052 + (length) - 0.150} 0 0.2" rpy="0 0 0" parent="shoulder_pitch_motor" child="elbow_motor" axis="0 1 0" l="-1.9880391011" u="1.97730123558" v="1.0"/>
   <xacro:Revjoint id="wrist_yaw" trans=" 0.015 -0.005 0.278" rpy="0 0 0" parent="elbow_motor" child="wrist_yaw_motor" axis="0 0 1" l="-2.617" u="2.617" v="1.0"/>

Commit message: urdf reverted back. Updated gripper.py

File: src/mobile_manipulator/model/mobile_manipulator.urdf (robot description, URDF)
Before this commit: robot mobile_manipulator, 9 links, 8 joints
Joints:
- joint shoulder_yaw: origin xyz=0.0965 -0.003 0.26 rpy=0 0 0 -> xyz=0.1765 -0.003 0.26 rpy=0 0 0

File: src/mobile_manipulator/model/mobile_manipulator.xacro (robot description, xacro)
@@ -293,7 +293,7 @@
   </link>
   <link name="shoulder_yaw_motor">
-    <xacro:shoulder_yaw_inertial trans="0.05 -0.02 0.1715" rpy="0 0 0 "/>
-    <xacro:shoulder_yaw_visual trans="0.05 -0.02 0.1715" rpy="0 0 0 "/>
-    <xacro:shoulder_yaw_collision trans="0.05 -0.02 0.1715" rpy="0 0 0"/>
+    <xacro:shoulder_yaw_inertial trans="0.13 -0.02 0.1715" rpy="0 0 0 "/>
+    <xacro:shoulder_yaw_visual trans="0.13 -0.02 0.1715" rpy="0 0 0 "/>
+    <xacro:shoulder_yaw_collision trans="0.13 -0.02 0.1715" rpy="0 0 0"/>
   </link>
   <link name="shoulder_bracket">
@@ -334,5 +334,5 @@
  <!-- JOINTS -->
    <xacro:FxdJoint id="bot_joint" trans="0 0 0" rpy="0 0 0" parent="bot" child="shoulder_yaw_motor"/>
-  <xacro:Revjoint id="shoulder_yaw" trans="0.0965 -0.003 0.26" rpy="0 0 0" parent="shoulder_yaw_motor" child="shoulder_bracket" axis="0 0 1" l="-3.14" u="3.14" v="1.0"/>
+  <xacro:Revjoint id="shoulder_yaw" trans="0.1765 -0.003 0.26" rpy="0 0 0" parent="shoulder_yaw_motor" child="shoulder_bracket" axis="0 0 1" l="-3.14" u="3.14" v="1.0"/>
   <xacro:Revjoint id="shoulder_pitch" trans="0.0 0.010 0.040" rpy="0 0 0.0" parent="shoulder_bracket" child="shoulder_pitch_motor" axis="0 1 0" l="-1.59" u="1.97423327401" v="1.0"/>
   <xacro:Revjoint id="elbow" trans="${0.052 + (length) - 0.150} 0 0.2" rpy="0 0 0" parent="shoulder_pitch_motor" child="elbow_motor" axis="0 1 0" l="-1.9880391011" u="1.97730123558" v="1.0"/>
@@ -342,2 +342,3 @@
   <xacro:FxdJoint id="end_eff_joint" trans="0.20 0 0.02" rpy="0 0 0" parent="wrist_roll_motor" child="end_effector_link"/>
 </robot>
+<!-- 0.0965 -->

Commit message: Urdf changed

File: src/mobile_manipulator/model/mobile_manipulator.urdf (robot description, URDF)
Before this commit: robot mobile_manipulator, 9 links, 8 joints
Joints:
- joint shoulder_yaw: origin xyz=0.1765 -0.003 0.26 rpy=0 0 0 -> xyz=0.0965 -0.003 0.26 rpy=0 0 0

File: src/mobile_manipulator/model/mobile_manipulator.xacro (robot description, xacro)
@@ -293,7 +293,7 @@
   </link>
   <link name="shoulder_yaw_motor">
-    <xacro:shoulder_yaw_inertial trans="0.13 -0.02 0.1715" rpy="0 0 0 "/>
-    <xacro:shoulder_yaw_visual trans="0.13 -0.02 0.1715" rpy="0 0 0 "/>
-    <xacro:shoulder_yaw_collision trans="0.13 -0.02 0.1715" rpy="0 0 0"/>
+    <xacro:shoulder_yaw_inertial trans="0.05 -0.02 0.1715" rpy="0 0 0 "/>  <!--0.13-->
+    <xacro:shoulder_yaw_visual trans="0.05 -0.02 0.1715" rpy="0 0 0 "/>
+    <xacro:shoulder_yaw_collision trans="0.05 -0.02 0.1715" rpy="0 0 0"/>
   </link>
   <link name="shoulder_bracket">
@@ -334,5 +334,5 @@
  <!-- JOINTS -->
    <xacro:FxdJoint id="bot_joint" trans="0 0 0" rpy="0 0 0" parent="bot" child="shoulder_yaw_motor"/>
-  <xacro:Revjoint id="shoulder_yaw" trans="0.1765 -0.003 0.26" rpy="0 0 0" parent="shoulder_yaw_motor" child="shoulder_bracket" axis="0 0 1" l="-3.14" u="3.14" v="1.0"/>
+  <xacro:Revjoint id="shoulder_yaw" trans="0.0965 -0.003 0.26" rpy="0 0 0" parent="shoulder_yaw_motor" child="shoulder_bracket" axis="0 0 1" l="-3.14" u="3.14" v="1.0"/>
   <xacro:Revjoint id="shoulder_pitch" trans="0.0 0.010 0.040" rpy="0 0 0.0" parent="shoulder_bracket" child="shoulder_pitch_motor" axis="0 1 0" l="-1.59" u="1.97423327401" v="1.0"/>
   <xacro:Revjoint id="elbow" trans="${0.052 + (length) - 0.150} 0 0.2" rpy="0 0 0" parent="shoulder_pitch_motor" child="elbow_motor" axis="0 1 0" l="-1.9880391011" u="1.97730123558" v="1.0"/>
@@ -342,3 +342,3 @@
   <xacro:FxdJoint id="end_eff_joint" trans="0.20 0 0.02" rpy="0 0 0" parent="wrist_roll_motor" child="end_effector_link"/>
 </robot>
-<!-- 0.0965 -->
+<!-- 0.1765 -->

Commit message: Backup commit with old urdf & broadcast

File: src/mobile_manipulator/model/mobile_manipulator.urdf (robot description, URDF)
Before this commit: robot mobile_manipulator, 9 links, 8 joints
Joints:
- joint shoulder_yaw: origin xyz=0.0965 -0.003 0.26 rpy=0 0 0 -> xyz=0.1765 -0.003 0.26 rpy=0 0 0
